File: Switch Matrix.kicad_sch (KiCad schematic)
At the start: 142 parts

Commit message: wip: matrix scheme refactored
Parts:
- added D_A1, D_D1, D_END1, D_F1, D_G1, D_H1, D_HELP1, D_J1, D_K1, D_L1, D_LINE1, D_QUOTE1, D_RETURN1, D_S1, D_SEMICOLON1, D_STATUS1, D_THUMB_DOWN1, D_THUMB_UP1: D, Diode_SMD:D_1210_3225Metric_Pad1.42x2.65mm_HandSolder, symbol Device:D
- added D_COLON1, D_EIGHT1, D_EQ1, D_FIVE1, D_FOUR1, D_LCURVEP1, D_MINUS1, D_NINE1, D_ONE1, D_RCURVEP1, D_SEVEN1, D_SIX1, D_THREE1, D_TWO1, D_ZERO1: D, symbol Device:D
- added S_A1: A, Button_Switch_Keyboard:SW_MX_1U, symbol Space_Cadet_Button_Switches:SWK
- added S_D1: D, Button_Switch_Keyboard:SW_MX_1U, symbol Space_Cadet_Button_Switches:SWK
- added S_EIGHT1: EIGHT, Button_Switch_Keyboard:SW_MX_1U, symbol Space_Cadet_Button_Switches:SWK
- added S_END1: END1, Button_Switch_Keyboard:SW_MX_2U, symbol Space_Cadet_Button_Switches:SWK
- added S_EQ1: EQ, Button_Switch_Keyboard:SW_MX_1U, symbol Space_Cadet_Button_Switches:SWK
- added S_F1: F, Button_Switch_Keyboard:SW_MX_1U, symbol Space_Cadet_Button_Switches:SWK
- added S_FIVE1: FIVE, Button_Switch_Keyboard:SW_MX_1U, symbol Space_Cadet_Button_Switches:SWK
- added S_FOUR1: FOUR, Button_Switch_Keyboard:SW_MX_1U, symbol Space_Cadet_Button_Switches:SWK
- added S_G1: G, Button_Switch_Keyboard:SW_MX_1U, symbol Space_Cadet_Button_Switches:SWK
- added S_H1: H, Button_Switch_Keyboard:SW_MX_1U, symbol Space_Cadet_Button_Switches:SWK
- added S_HELP1: HELP, Button_Switch_Keyboard:SW_MX_2U, symbol Space_Cadet_Button_Switches:SWK
- added S_J1: J, Button_Switch_Keyboard:SW_MX_1U, symbol Space_Cadet_Button_Switches:SWK
- added S_K1: K, Button_Switch_Keyboard:SW_MX_1U, symbol Space_Cadet_Button_Switches:SWK
- added S_L1: L, Button_Switch_Keyboard:SW_MX_1U, symbol Space_Cadet_Button_Switches:SWK
- added S_LCURVEP1: LCURVEP, Button_Switch_Keyboard:SW_MX_1U, symbol Space_Cadet_Button_Switches:SWK
- added S_LINE1: LINE, Button_Switch_Keyboard:SW_MX_1U, symbol Space_Cadet_Button_Switches:SWK
- added S_MINUS1: MINUS, Button_Switch_Keyboard:SW_MX_1U, symbol Space_Cadet_Button_Switches:SWK
- added S_NINE1: NINE, Button_Switch_Keyboard:SW_MX_1U, symbol Space_Cadet_Button_Switches:SWK
- added S_ONE1: COLON, Button_Switch_Keyboard:SW_MX_1U, symbol Space_Cadet_Button_Switches:SWK
- added S_ONE1: ONE, Button_Switch_Keyboard:SW_MX_1U, symbol Space_Cadet_Button_Switches:SWK
- added S_QUOTE1: QUOTE, Button_Switch_Keyboard:SW_MX_1U, symbol Space_Cadet_Button_Switches:SWK
- added S_RCURVEP1: RCURVEP, Button_Switch_Keyboard:SW_MX_1U, symbol Space_Cadet_Button_Switches:SWK
- added S_RETURN1: RETURN, Button_Switch_Keyboard:SW_MX_1U, symbol Space_Cadet_Button_Switches:SWK
- added S_S1: S, Button_Switch_Keyboard:SW_MX_1U, symbol Space_Cadet_Button_Switches:SWK
- added S_SEMICOLON1: SEMICOLON, Button_Switch_Keyboard:SW_MX_1U, symbol Space_Cadet_Button_Switches:SWK
- added S_SEVEN1: SEVEN, Button_Switch_Keyboard:SW_MX_1U, symbol Space_Cadet_Button_Switches:SWK
- added S_SIX1: SIX, Button_Switch_Keyboard:SW_MX_1U, symbol Space_Cadet_Button_Switches:SWK
- added S_STATUS1: STATUS, Button_Switch_Keyboard:SW_MX_2U, symbol Space_Cadet_Button_Switches:SWK
- added S_THREE1: THREE, Button_Switch_Keyboard:SW_MX_1U, symbol Space_Cadet_Button_Switches:SWK
- added S_THUMB_DOWN1: THUMB_DOWN, Button_Switch_Keyboard:SW_MX_1U, symbol Space_Cadet_Button_Switches:SWK
- added S_THUMB_UP1: THUMB_UP, Button_Switch_Keyboard:SW_MX_1U, symbol Space_Cadet_Button_Switches:SWK
- added S_TWO1: TWO, Button_Switch_Keyboard:SW_MX_1U, symbol Space_Cadet_Button_Switches:SWK
- added S_ZERO1: ZERO, Button_Switch_Keyboard:SW_MX_1U, symbol Space_Cadet_Button_Switches:SWK
- S_ALTMODE1: renamed from S_ALT_MODE1; value ALT_MODE_1 -> ALTMODE
- S_BACKSLASH1: renamed from S_SLASH1; value SLASH_1 -> BACKSLASH
- S_BACKTICK1: renamed from S_QUOTE2; value QUOTE_2 -> BACKTICK
- S_BREAK1: value BREAK_1 -> BREAK
- S_CALL1: value CALL_1 -> CALL
- S_CLEAR_INPUT1: value CLEAR_INPUT_1 -> CLEAR_INPUT
- S_CLEAR_SCREEN1: value CLEAR_SCREEN_1 -> CLEAR_SCREEN
- S_DELETE1: value DELETE_1 -> DELETE
- S_DOT1: renamed from S_POINT1; value POINT -> DOT
- S_E1: value E_1 -> E
- S_HOLD_OUTPUT1: value HOLD_OUTPUT_1 -> HOLD_OUTPUT
- S_I_1: value I_1 -> I
- S_LEFT_ALT1: renamed from S_L_ALT1; value L_ALT -> LEFT_ALT
- S_LGREEK1: renamed from S_GREEK1; value GREEK -> LEFT_GREEK
- S_LMETA1: renamed from S_META1; value META -> LEFT_META
- S_LPAREN1: renamed from S_O_PRTHS1; value (_1 -> LPAREN
- S_NETWORK1: renamed from R2C1; value NETWORK_1 -> NETWORK
- S_O1: value O_1 -> O
- S_OVER_STRIKE1: value OVER_STRIKE_1 -> OVER_STRIKE
- S_P1: value P_1 -> P
- S_Q1: value Q_1 -> Q
- S_QUOTE1: value QUOTE_1 -> QUOTE
- S_R1: value R_1 -> R
- S_RESUME1: value RESUME_1 -> RESUME
- S_RIGHT_ALT1: renamed from S_L_ALT17; value L_ALT -> RIGHT_ALT
- S_ROM_FOUR1: renamed from S_ROM4; value ROM_4 -> ROM_THREE
- S_ROM_ONE1: renamed from S_ROM_1; value ROM_1 -> ROM_ONE
- S_ROM_THREE1: renamed from S_ROM3; value ROM_3 -> ROM_THREE
- S_ROM_TWO1: renamed from S_ROM_2; value ROM_2 -> ROM_TWO
- S_RPAREN1: renamed from S_C_PRTHS1; value )_1 -> RPAREN
- S_RUBOUT1: renamed from S_RUB_OUT1; value RUB_OUT_1 -> RUBOUT
- S_SLASH1: renamed from S_QUESTION1; value QUESTION -> SLASH
- S_STOP_OUTPUT1: value STOP_OUTPUT_1 -> STOP_OUTPUT
- S_T1: value T1 -> T
- S_TAB1: value TAB_1 -> TAB
- S_TERMINAL1: value TERMINAL_1 -> TERMINAL
- S_THUMB_LEFT1: renamed from S_H_LEFT1; value H_LEFT_1 -> THUMB_LEFT
- S_THUMB_RIGHT1: renamed from S_H_RIGHT1; value H_RIGHT_1 -> THUMB_RIGHT
- S_U1: value U_1 -> U
- S_W1: value W_1 -> W
- S_Y1: value Y_1 -> Y
- renumbered D_ABORT18 to D_ABORT1, D_ALT_LOCK17 to D_ALTLOCK1, D_ALT_MODE1 to D_ALTMODE1, D_B18 to D_B1, D_SLASH18 to D_BACKSLASH1, D_QUOTE2 to D_BACKTICK1, D_C18 to D_C1, D_CLEAR_INPUT18 to D_CLEAR_INPUT, D_L_CTRL17 to D_CTRL1, D_POINT1 to D_DOT1, D_L_ALT1 to D_LEFT_ALT1, D_LEFT_SPACE1 to D_LEFT_SPC1, D_GREEK1 to D_LGREEK1, D_L_HYPER1 to D_LHYPER1, D_L_META1 to D_LMETA1, D_O_PRTHS1 to D_LPAREN1, D_L_SHIFT1 to D_LSHIFT1, D_L_SUPER1 to D_LSUPER1, D_M17 to D_M1, D_N19 to D_N1, D_O20 to D_O1, D_QUOTE1 to D_QUOTE_MOD, D_R_CTRL1 to D_RCTRL1, D_R_GREEK17 to D_RGREEK1, D_R_HYPER1 to D_RHYPER1, D_L_ALT17 to D_RIGHT_ALT1, D_RIGHT_SPACE17 to D_RIGHT_SPACE1, D_R_META1 to D_RMETA1, D_ROM_4 to D_ROM_FOUR1, D_ROM_1 to D_ROM_ONE1, D_ROM_3 to D_ROM_THREE1, D_ROM_2 to D_ROM_TWO1, D_C_PRTHS18 to D_RPAREN1, D_R_SHIFT17 to D_RSHIFT1, D_R_SUPER1 to D_RSUPER1, D_RUB_OUT1 to D_RUBOUT1, D_QUESTION1 to D_SLASH1, D_H_LEFT1 to D_THUMB_LEFT1, D_H_RIGHT1 to D_THUMB_RIGHT1, D_TOP17 to D_TOP1, D_V18 to D_V1, D_X17 to D_X1, S_A_LOCK17 to S_ALTLOCK1, S_B18 to S_B1, S_C18 to S_C1, S_C_LOCK1 to S_CAPSLOCK1, S_L_CTRL1 to S_CTRL1, S_L_SPC1 to S_LEFT_SPC1, S_L_HYPER1 to S_LHYPER1, S_L_SHIFT1 to S_LSHIFT1, S_L_SUPER1 to S_LSUPER1, S_N17 to S_N1, S_R_CTRL17 to S_RCTRL1, S_R_GREEK17 to S_RGREEK1, S_R_HYPER17 to S_RHYPER1, S_RIGHT_SPACE17 to S_RIGHT_SPACE1, S_R_META1 to S_RMETA1, S_R_SHIFT17 to S_RSHIFT1, S_R_SUPER1 to S_RSUPER1, S_TOP17 to S_TOP1, S_V18 to S_V1, S_X17 to S_X1
Connections:
- net COL16: no longer S_LKM1.2 (out)
- net ROW2: no longer D_ROM_THREE1.1 (K)
- net ROW5: no longer D_LKM1.1 (K), D_RCTRL1.1 (K), D_RIGHT_ALT1.1 (K), D_RMETA1.1 (K)
- net at D_BREAK1.2 (A): no longer S_BREAK1.2 (out)
- net at S_ROM_ONE1.2 (out): no longer D_ROM_ONE1.2 (A)
- net at D_RESUME1.2 (A): no longer S_RESUME1.2 (out)
- net at S_CALL1.2 (out): no longer D_CALL1.2 (A)
- net at D_HOLD_OUTPUT1.2 (A): no longer S_HOLD_OUTPUT1.2 (out)
- net at S_STOP_OUTPUT1.2 (out): no longer D_STOP_OUTPUT1.2 (A)
- net at D_ROM_TWO1.2 (A): no longer S_ROM_TWO1.2 (out)
- net at S_DELETE1.2 (out): no longer D_DELETE1.2 (A)
- net at S_OVER_STRIKE1.2 (out): no longer D_OVER_STRIKE1.2 (A)
- net at S_NETWORK1.2 (out): no longer D_NETWORK1.2 (A)
- net at S_MACRO1.2 (out): no longer D_MACRO1.2 (A)
- net at D_QUOTE_MOD.2 (A): no longer S_QUOTE1.2 (out)
- net at D_SYSTEM1.2 (A): no longer S_SYSTEM1.2 (out)
- net at D_CLEAR_INPUT.2 (A): no longer S_CLEAR_INPUT1.2 (out)
- net at S_TERMINAL1.2 (out): no longer D_TERMINAL1.2 (A)
- net at D_CLEAR_SCREEN1.2 (A): no longer S_CLEAR_SCREEN1.2 (out)
- net at S_ABORT18.2 (out): no longer D_ABORT1.2 (A)
Other:
- moved on the sheet: D_ABORT1, D_ALTLOCK1, D_ALTMODE1, D_B1, D_BACKSLASH1, D_BACKTICK1, D_BREAK1, D_C1, D_CALL1, D_CAPS_LOCK1, D_CLEAR_INPUT, D_CLEAR_SCREEN1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

Commit message: add some conventional modifiers
Parts:
- added D_LEFT_SPC17: D, Diode_SMD:D_1210_3225Metric_Pad1.42x2.65mm_HandSolder, symbol Device:D
- added S_LEFT_SPC17: LEFT_SPACE, Button_Switch_Keyboard:SW_MX_1U, symbol Space_Cadet_Button_Switches:SWK
- S_FN: renamed from S_LEFT_SPC1; value LEFT_SPACE -> FN
- renumbered D_LEFT_SPC1 to D_FN
Other:
- moved on the sheet: D_RCTRL1, D_RESUME1, D_RIGHT_ALT1, D_RIGHT_SPACE1, S_RCTRL1, S_RESUME1, S_RIGHT_ALT1, S_RIGHT_SPACE1

Commit message: RP2040 added
Parts:
- D_A1, D_ABORT1, D_ALTLOCK1, D_ALTMODE1, D_B1, D_BACKSLASH1, D_BACKTICK1, D_BREAK1, D_C1, D_CALL1, D_CAPS_LOCK1, D_CLEAR_SCREEN1, D_COMMA1, D_CTRL1, D_D1, D_DELETE1, D_DOT1, D_E1, D_END1, D_F1, D_G1, D_H1, D_HELP1, D_HOLD_OUTPUT1, D_I_1, D_J1, D_K1, D_L1, D_LEFT_ALT1, D_LEFT_SPC17, D_LGREEK1, D_LHYPER1, D_LINE1, D_LKM1, D_LMETA1, D_LPAREN1, D_LSHIFT1, D_LSUPER1, D_M1, D_MACRO1, D_MODE_LOCK1, D_N1, D_NETWORK1, D_O1, D_OVER_STRIKE1, D_P1, D_Q1, D_QUOTE1, D_R1, D_RCTRL1, D_REPEAT1, D_RESUME1, D_RETURN1, D_RGREEK1, D_RHYPER1, D_RIGHT_ALT1, D_RIGHT_SPACE1, D_RMETA1, D_ROM_FOUR1, D_ROM_ONE1, D_ROM_THREE1, D_ROM_TWO1, D_RPAREN1, D_RSHIFT1, D_RSUPER1, D_RUBOUT1, D_S1, D_SEMICOLON1, D_SLASH1, D_STATUS1, D_STOP_OUTPUT1, D_SYSTEM1, D_T1, D_TAB1, D_TERMINAL1, D_THUMB_DOWN1, D_THUMB_LEFT1, D_THUMB_RIGHT1, D_THUMB_UP1, D_U1, D_V1, D_W1, D_X1, D_Y1, D_Z1: footprint Diode_SMD:D_1210_3225Metric_Pad1.42x2.65mm_HandSolder -> Diode_SMD:D_SOD-123; symbol Device:D -> Device:D_Small
- D_CLEAR_INPUT1: renamed from D_CLEAR_INPUT; footprint Diode_SMD:D_1210_3225Metric_Pad1.42x2.65mm_HandSolder -> Diode_SMD:D_SOD-123; symbol Device:D -> Device:D_Small
- D_COLON1, D_EIGHT1, D_EQ1, D_FIVE1, D_FOUR1, D_LCURVEP1, D_MINUS1, D_NINE1, D_ONE1, D_RCURVEP1, D_SEVEN1, D_SIX1, D_THREE1, D_TWO1, D_ZERO1: footprint (none) -> Diode_SMD:D_SOD-123; symbol Device:D -> Device:D_Small
- D_FN1: renamed from D_FN; footprint Diode_SMD:D_1210_3225Metric_Pad1.42x2.65mm_HandSolder -> Diode_SMD:D_SOD-123; symbol Device:D -> Device:D_Small
- D_LTOP1, D_RTOP1: renamed from D_TOP1; footprint Diode_SMD:D_1210_3225Metric_Pad1.42x2.65mm_HandSolder -> Diode_SMD:D_SOD-123; symbol Device:D -> Device:D_Small
- D_QUOTE_MOD1: renamed from D_QUOTE_MOD; footprint Diode_SMD:D_1210_3225Metric_Pad1.42x2.65mm_HandSolder -> Diode_SMD:D_SOD-123; symbol Device:D -> Device:D_Small
- S_LTOP1: renamed from S_TOP1; value TOP -> LEFT_TOP
- S_QUOTE_MOD1: renamed from S_QUOTE1; value QUOTE -> QUOTE_MOD
- S_RTOP1: renamed from S_TOP1; value TOP -> RIGHT_TOP
- renumbered S_ONE1 to S_COLON1, S_FN to S_FN1

Commit message: deps
Parts:
- S_A1: dep (none) -> S_RUBOUT1
- S_ABORT18: dep (none) -> S_STOP_OUTPUT1
- S_ALTLOCK1: dep (none) -> S_REPEAT1
- S_ALTMODE1: dep (none) -> S_M_LOCK1
- S_B1: dep (none) -> S_V1
- S_BACKSLASH1: dep (none) -> S_BACKTICK1
- S_BACKTICK1: dep (none) -> S_RPAREN1
- S_BREAK1: dep (none) -> S_ABORT18
- S_C1: dep (none) -> S_X1
- S_CALL1: dep (none) -> S_RESUME1
- S_CLEAR_INPUT1: dep (none) -> S_OVER_STRIKE1
- S_CLEAR_SCREEN1: dep (none) -> S_CLEAR_INPUT1
- S_COLON1: dep (none) -> S_SYSTEM1
- S_COMMA1: dep (none) -> S_M17
- S_CTRL1: dep (none) -> S_LMETA1
- S_D1: dep (none) -> S_S1
- S_DELETE1: dep (none) -> S_BACKSLASH1
- S_DOT1: dep (none) -> S_COMMA1
- S_E1: dep (none) -> S_W1
- S_EIGHT1: dep (none) -> S_SEVEN1
- S_END1: dep (none) -> S_LINE1
- S_EQ1: dep (none) -> S_MINUS1
- S_F1: dep (none) -> S_D1
- S_FIVE1: dep (none) -> S_FOUR1
- S_FN1: dep (none) -> S_LEFT_ALT1
- S_FOUR1: dep (none) -> S_THREE1
- S_G1: dep (none) -> S_F1
- S_H1: dep (none) -> S_G1
- S_HELP1: dep (none) -> S_END1
- S_HOLD_OUTPUT1: dep (none) -> S_CLEAR_SCREEN1
- S_I_1: dep (none) -> S_U1
- S_J1: dep (none) -> S_H1
- S_K1: dep (none) -> S_J1
- S_L1: dep (none) -> S_K1
- S_LCURVEP1: dep (none) -> S_EQ1
- S_LEFT_ALT1: dep (none) -> S_CTRL1
- S_LEFT_SPC17: dep (none) -> S_FN1
- S_LGREEK1: dep (none) -> S_LTOP1
- S_LINE1: dep (none) -> S_RETURN1
- S_LKM1: dep (none) -> S_RIGHT_SPACE1
- S_LMETA1: dep (none) -> S_LSUPER1
- S_LPAREN1: dep (none) -> S_P1
- S_LSHIFT1: dep (none) -> S_LGREEK1
- S_LSUPER1: dep (none) -> S_LHYPER1
- S_LTOP1: dep (none) -> S_CAPSLOCK1
- S_M17: dep (none) -> S_N1
- S_MINUS1: dep (none) -> S_ZERO1
- S_N1: dep (none) -> S_B1
- S_NETWORK1: dep (none) -> S_ROM_FOUR1
- S_O1: dep (none) -> S_I_1
- S_ONE1: dep (none) -> S_COLON1
- S_OVER_STRIKE1: dep (none) -> S_QUOTE_MOD1
- S_P1: dep (none) -> S_O1
- S_Q1: dep (none) -> S_TAB1
- S_QUOTE1: dep (none) -> S_SEMICOLON1
- S_QUOTE_MOD1: dep (none) -> S_TERMINAL1
- S_R1: dep (none) -> S_E1
- S_RCTRL1: dep (none) -> S_RIGHT_ALT1
- S_RCURVEP1: dep (none) -> S_LCURVEP1
- S_REPEAT1: dep (none) -> S_RTOP1
- S_RESUME1: dep (none) -> S_BREAK1
- S_RETURN1: dep (none) -> S_QUOTE1
- S_RGREEK1: dep (none) -> S_RSHIFT1
- S_RHYPER1: dep (none) -> S_RSUPER1
- S_RIGHT_ALT1: dep (none) -> S_LKM1
- S_RIGHT_SPACE1: dep (none) -> S_LEFT_SPC17
- S_RMETA1: dep (none) -> S_RCTRL1
- S_ROM_FOUR1: dep (none) -> S_ROM_THREE1
- S_ROM_TWO1: dep (none) -> S_ROM_ONE1
- S_RPAREN1: dep (none) -> S_LPAREN1
- S_RSHIFT1: dep (none) -> S_SLASH1
- S_RSUPER1: dep (none) -> S_RMETA1
- S_RTOP1: dep (none) -> S_RGREEK1
- S_RUBOUT1: dep (none) -> S_ALTMODE1
- S_S1: dep (none) -> S_A1
- S_SEMICOLON1: dep (none) -> S_L1
- S_SEVEN1: dep (none) -> S_SIX1
- S_SIX1: dep (none) -> S_FIVE1
- S_SLASH1: dep (none) -> S_DOT1
- S_STATUS1: dep (none) -> S_RCURVEP1
- S_STOP_OUTPUT1: dep (none) -> S_HOLD_OUTPUT1
- S_SYSTEM1: dep (none) -> S_ROM_TWO1
- S_T1: dep (none) -> S_R1
- S_TAB1: dep (none) -> S_NETWORK1
- S_TERMINAL1: dep (none) -> S_MACRO1
- S_THREE1: dep (none) -> S_TWO1
- S_THUMB_DOWN1: dep (none) -> S_THUMB_UP1
- S_THUMB_LEFT1: dep (none) -> S_DELETE1
- S_THUMB_RIGHT1: dep (none) -> S_THUMB_LEFT1
- S_THUMB_UP1: dep (none) -> S_STATUS1
- S_TWO1: dep (none) -> S_ONE1
- S_U1: dep (none) -> S_Y1
- S_V1: dep (none) -> S_C1
- S_W1: dep (none) -> S_Q1
- S_X1: dep (none) -> S_Z1
- S_Y1: dep (none) -> S_T1
- S_Z1: dep (none) -> S_LSHIFT1
- S_ZERO1: dep (none) -> S_NINE1
Other:
- moved on the sheet: S_THUMB_DOWN1

Commit message: wip: dag building, prepare for replace coords
Parts:
- S_NINE1: dep (none) -> S_EIGHT1
Changed lines of the file:
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@@
+			)
+		)
+		(property "dep" "S_EIGHT1"
+			(at 279.4 85.09 0)
+			(effects
+				(font
+					(size 1.27 1.27)
+				)
+				(hide yes)
 			)
 		)

Commit message: wip: fix units, added commets, added todos
Parts:
- S_B1, S_C1, S_M17, S_N1, S_ROM_TWO1, S_V1, S_X1, S_Z1: footprint Button_Switch_Keyboard:SW_MX_2U -> Button_Switch_Keyboard:SW_MX_1U
- S_ROM_FOUR1: value ROM_THREE -> ROM_FOUR
Changed lines of the file:
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@@
 			)
 		)
-		(property "Footprint" "Button_Switch_Keyboard:SW_MX_2U"
+		(property "Footprint" "Button_Switch_Keyboard:SW_MX_1U"
 			(at 242.824 153.67 0)
 			(effects
@@
 			)
 		)
-		(property "Footprint" "Button_Switch_Keyboard:SW_MX_2U"
+		(property "Footprint" "Button_Switch_Keyboard:SW_MX_1U"
 			(at 223.774 153.67 0)
 			(effects
@@
 			)
 		)
-		(property "Footprint" "Button_Switch_Keyboard:SW_MX_2U"
+		(property "Footprint" "Button_Switch_Keyboard:SW_MX_1U"
 			(at 71.374 87.63 0)
 			(effects
@@
 			)
 		)
-		(property "Value" "ROM_THREE"
+		(property "Value" "ROM_FOUR"
 			(at 68.326 106.045 0)
 			(effects
@@
 			)
 		)
-		(property "Footprint" "Button_Switch_Keyboard:SW_MX_2U"
+		(property "Footprint" "Button_Switch_Keyboard:SW_MX_1U"
 			(at 128.524 153.67 0)
 			(effects
@@
 			)
 		)
-		(property "Footprint" "Button_Switch_Keyboard:SW_MX_2U"
+		(property "Footprint" "Button_Switch_Keyboard:SW_MX_1U"
 			(at 185.674 153.67 0)
 			(effects
@@
 			)
 		)
-		(property "Footprint" "Button_Switch_Keyboard:SW_MX_2U"
+		(property "Footprint" "Button_Switch_Keyboard:SW_MX_1U"
 			(at 204.724 153.67 0)
 			(effects
@@
 			)
 		)
-		(property "Footprint" "Button_Switch_Keyboard:SW_MX_2U"
+		(property "Footprint" "Button_Switch_Keyboard:SW_MX_1U"
 			(at 166.624 153.67 0)
 			(effects
@@
 			)
 		)
-		(property "Footprint" "Button_Switch_Keyboard:SW_MX_2U"
+		(property "Footprint" "Button_Switch_Keyboard:SW_MX_1U"
 			(at 147.574 153.67 0)
 			(effects

Commit message: ready replacer
Parts:
- S_COMMA1, S_DOT1, S_SLASH1: footprint Button_Switch_Keyboard:SW_MX_2U -> Button_Switch_Keyboard:SW_MX_1U
Changed lines of the file:
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@@
 			)
 		)
-		(property "Footprint" "Button_Switch_Keyboard:SW_MX_2U"
+		(property "Footprint" "Button_Switch_Keyboard:SW_MX_1U"
 			(at 280.924 153.67 0)
 			(effects
@@
 			)
 		)
-		(property "Footprint" "Button_Switch_Keyboard:SW_MX_2U"
+		(property "Footprint" "Button_Switch_Keyboard:SW_MX_1U"
 			(at 261.874 153.67 0)
 			(effects
@@
 			)
 		)
-		(property "Footprint" "Button_Switch_Keyboard:SW_MX_2U"
+		(property "Footprint" "Button_Switch_Keyboard:SW_MX_1U"
 			(at 299.974 153.67 0)
 			(effects

Commit message: wip: sch fixes
Parts:
- S_EQ1, S_MINUS1: footprint Button_Switch_Keyboard:SW_MX_1U -> Button_Switch_Keyboard:SW_MX_1.45U
- S_RUBOUT1: footprint Button_Switch_Keyboard:SW_MX_2U -> Button_Switch_Keyboard:SW_MX_1.45U
- S_TAB1: footprint Button_Switch_Keyboard:SW_MX_2U -> Button_Switch_Keyboard:SW_MX_1.25U
Changed lines of the file:
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@@
 			)
 		)
-		(property "Footprint" "Button_Switch_Keyboard:SW_MX_2U"
+		(property "Footprint" "Button_Switch_Keyboard:SW_MX_1.25U"
 			(at 109.474 107.95 0)
 			(effects
@@
 			)
 		)
-		(property "Footprint" "Button_Switch_Keyboard:SW_MX_2U"
+		(property "Footprint" "Button_Switch_Keyboard:SW_MX_1.45U"
 			(at 109.474 130.81 0)
 			(effects
@@
 			)
 		)
-		(property "Footprint" "Button_Switch_Keyboard:SW_MX_1U"
+		(property "Footprint" "Button_Switch_Keyboard:SW_MX_1.45U"
 			(at 338.328 87.63 0)
 			(effects
@@
 			)
 		)
-		(property "Footprint" "Button_Switch_Keyboard:SW_MX_1U"
+		(property "Footprint" "Button_Switch_Keyboard:SW_MX_1.45U"
 			(at 319.278 87.63 0)
 			(effects
