File: Switch Matrix.kicad_sch (KiCad schematic)
At the start: 210 parts

Commit message: wip: new buttons
Parts:
- S_BACKSLASH1: footprint Button_Switch_Keyboard:SW_MX_1U -> Button_Switch_Keyboard:SW_MX_1.5U
- S_CTRL1, S_LEFT_ALT1, S_LGREEK1, S_LHYPER1, S_LMETA1, S_LSUPER1, S_LTOP1, S_RCTRL1, S_REPEAT1, S_RGREEK1, S_RHYPER1, S_RIGHT_ALT1, S_RMETA1, S_RSUPER1, S_RTOP1, S_TAB1: footprint Button_Switch_Keyboard:SW_MX_1.25U -> Button_Switch_Keyboard:SW_MX_1.5U
- S_EQ1, S_MINUS1: footprint Button_Switch_Keyboard:SW_MX_1.45U -> Button_Switch_Keyboard:SW_MX_1.5U
- S_LEFT_SPC17, S_RIGHT_SPACE1: footprint Button_Switch_Keyboard:SW_MX_1U -> Button_Switch_Keyboard:SW_MX_3U
- S_LINE1: footprint Button_Switch_Keyboard:SW_MX_1U -> Button_Switch_Keyboard:SW_MX_1.25U
- S_RETURN1: footprint Button_Switch_Keyboard:SW_MX_1U -> Button_Switch_Keyboard:SW_MX_2U
- S_RUBOUT1: footprint Button_Switch_Keyboard:SW_MX_1.45U -> Button_Switch_Keyboard:SW_MX_1.75U
Changed lines of the file:
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@@
 			)
 		)
-		(property "Footprint" "Button_Switch_Keyboard:SW_MX_1.25U"
+		(property "Footprint" "Button_Switch_Keyboard:SW_MX_1.5U"
 			(at 71.374 175.26 0)
 			(effects
@@
 			)
 		)
-		(property "Footprint" "Button_Switch_Keyboard:SW_MX_1.25U"
+		(property "Footprint" "Button_Switch_Keyboard:SW_MX_1.5U"
 			(at 433.324 175.26 0)
 			(effects
@@
 			)
 		)
-		(property "Footprint" "Button_Switch_Keyboard:SW_MX_1.25U"
+		(property "Footprint" "Button_Switch_Keyboard:SW_MX_1.5U"
 			(at 109.474 175.26 0)
 			(effects
@@
 			)
 		)
-		(property "Footprint" "Button_Switch_Keyboard:SW_MX_1.25U"
+		(property "Footprint" "Button_Switch_Keyboard:SW_MX_1.5U"
 			(at 71.374 153.67 0)
 			(effects
@@
 			)
 		)
-		(property "Footprint" "Button_Switch_Keyboard:SW_MX_1U"
+		(property "Footprint" "Button_Switch_Keyboard:SW_MX_3U"
 			(at 261.874 176.53 0)
 			(effects
@@
 			)
 		)
-		(property "Footprint" "Button_Switch_Keyboard:SW_MX_1.25U"
+		(property "Footprint" "Button_Switch_Keyboard:SW_MX_1.5U"
 			(at 109.474 107.95 0)
 			(effects
@@
 			)
 		)
-		(property "Footprint" "Button_Switch_Keyboard:SW_MX_1.25U"
+		(property "Footprint" "Button_Switch_Keyboard:SW_MX_1.5U"
 			(at 90.424 175.26 0)
 			(effects
@@
 			)
 		)
-		(property "Footprint" "Button_Switch_Keyboard:SW_MX_1.25U"
+		(property "Footprint" "Button_Switch_Keyboard:SW_MX_1.5U"
 			(at 376.174 175.26 0)
 			(effects
@@
 			)
 		)
-		(property "Footprint" "Button_Switch_Keyboard:SW_MX_1.25U"
+		(property "Footprint" "Button_Switch_Keyboard:SW_MX_1.5U"
 			(at 357.124 175.26 0)
 			(effects
@@
 			)
 		)
-		(property "Footprint" "Button_Switch_Keyboard:SW_MX_1.25U"
+		(property "Footprint" "Button_Switch_Keyboard:SW_MX_1.5U"
 			(at 52.324 175.26 0)
 			(effects
@@
 			)
 		)
-		(property "Footprint" "Button_Switch_Keyboard:SW_MX_1.25U"
+		(property "Footprint" "Button_Switch_Keyboard:SW_MX_1.5U"
 			(at 338.074 153.67 0)
 			(effects
@@
 			)
 		)
-		(property "Footprint" "Button_Switch_Keyboard:SW_MX_1.25U"
+		(property "Footprint" "Button_Switch_Keyboard:SW_MX_1.5U"
 			(at 90.424 153.67 0)
 			(effects
@@
 			)
 		)
-		(property "Footprint" "Button_Switch_Keyboard:SW_MX_1.45U"
+		(property "Footprint" "Button_Switch_Keyboard:SW_MX_1.75U"
 			(at 109.474 130.81 0)
 			(effects
@@
 			)
 		)
-		(property "Footprint" "Button_Switch_Keyboard:SW_MX_1.25U"
+		(property "Footprint" "Button_Switch_Keyboard:SW_MX_1.5U"
 			(at 395.478 152.654 0)
 			(effects
@@
 			)
 		)
-		(property "Footprint" "Button_Switch_Keyboard:SW_MX_1U"
+		(property "Footprint" "Button_Switch_Keyboard:SW_MX_1.25U"
 			(at 357.124 130.81 0)
 			(effects
@@
 			)
 		)
-		(property "Footprint" "Button_Switch_Keyboard:SW_MX_1.45U"
+		(property "Footprint" "Button_Switch_Keyboard:SW_MX_1.5U"
 			(at 338.328 87.63 0)
 			(effects
@@
 			)
 		)
-		(property "Footprint" "Button_Switch_Keyboard:SW_MX_1.25U"
+		(property "Footprint" "Button_Switch_Keyboard:SW_MX_1.5U"
 			(at 414.274 175.26 0)
 			(effects
@@
 			)
 		)
-		(property "Footprint" "Button_Switch_Keyboard:SW_MX_1U"
+		(property "Footprint" "Button_Switch_Keyboard:SW_MX_2U"
 			(at 338.074 130.81 0)
 			(effects
@@
 			)
 		)
-		(property "Footprint" "Button_Switch_Keyboard:SW_MX_1.45U"
+		(property "Footprint" "Button_Switch_Keyboard:SW_MX_1.5U"
 			(at 319.278 87.63 0)
 			(effects
@@
 			)
 		)
-		(property "Footprint" "Button_Switch_Keyboard:SW_MX_1.25U"
+		(property "Footprint" "Button_Switch_Keyboard:SW_MX_1.5U"
 			(at 414.528 152.654 0)
 			(effects
@@
 			)
 		)
-		(property "Footprint" "Button_Switch_Keyboard:SW_MX_1U"
+		(property "Footprint" "Button_Switch_Keyboard:SW_MX_3U"
 			(at 224.028 176.784 0)
 			(effects
@@
 			)
 		)
-		(property "Footprint" "Button_Switch_Keyboard:SW_MX_1.25U"
+		(property "Footprint" "Button_Switch_Keyboard:SW_MX_1.5U"
 			(at 128.524 175.26 0)
 			(effects
@@
 			)
 		)
-		(property "Footprint" "Button_Switch_Keyboard:SW_MX_1.25U"
+		(property "Footprint" "Button_Switch_Keyboard:SW_MX_1.5U"
 			(at 395.224 175.26 0)
 			(effects
@@
 			)
 		)
-		(property "Footprint" "Button_Switch_Keyboard:SW_MX_1U"
+		(property "Footprint" "Button_Switch_Keyboard:SW_MX_1.5U"
 			(at 376.174 107.95 0)
 			(effects

Commit message: wip: pcb+hypo
Parts:
- removed D_LEFT_SPC17: D, Diode_SMD:D_SOD-123, symbol Device:D_Small
- removed S_LEFT_SPC17: LEFT_SPACE, Button_Switch_Keyboard:SW_MX_3U, symbol Space_Cadet_Button_Switches:SWK
- added D_LEFT_SPACE1, D_LHYPO1, D_LKM201, D_PLUS1, D_RHYPO1: D, Diode_SMD:D_SOD-123, symbol Device:D_Small
- added S_LEFT_SPACE1: LEFT_SPACE, Button_Switch_Keyboard:SW_Cherry_MX_2.75u_PCB, symbol Space_Cadet_Button_Switches:SWK
- added S_LHYPO1: LEFT_HYPO, Button_Switch_Keyboard:SW_Cherry_MX_6.25u_PCB, symbol Space_Cadet_Button_Switches:SWK
- added S_LKM1: LKM, Button_Switch_Keyboard:SW_Cherry_MX_1.25u_PCB, symbol Space_Cadet_Button_Switches:SWK
- added S_PLUS1: PLUS, Button_Switch_Keyboard:SW_Cherry_MX_1.00u_PCB, symbol Space_Cadet_Button_Switches:SWK
- added S_RHYPO1: RIGHT_HYPO, Button_Switch_Keyboard:SW_Cherry_MX_6.25u_PCB, symbol Space_Cadet_Button_Switches:SWK
- S_A1, S_ALTLOCK1, S_B1, S_BACKTICK1, S_C1, S_CAPSLOCK1, S_COLON1, S_COMMA1, S_D1, S_DOT1, S_E1, S_EIGHT1, S_F1, S_FIVE1, S_FOUR1, S_G1, S_H1, S_I_1, S_J1, S_K1, S_L1, S_LCURVEP1, S_LPAREN1, S_M17, S_N1, S_NINE1, S_O1, S_ONE1, S_P1, S_Q1, S_QUOTE1, S_R1, S_RCURVEP1, S_ROM_FOUR1, S_ROM_ONE1, S_ROM_THREE1, S_ROM_TWO1, S_RPAREN1, S_S1, S_SEMICOLON1, S_SEVEN1, S_SIX1, S_SLASH1, S_T1, S_THREE1, S_THUMB_DOWN1, S_THUMB_LEFT1, S_THUMB_RIGHT1, S_THUMB_UP1, S_TWO1, S_U1, S_V1, S_W1, S_X1, S_Y1, S_Z1, S_ZERO1: footprint Button_Switch_Keyboard:SW_MX_1U -> Button_Switch_Keyboard:SW_Cherry_MX_1.00u_PCB
- S_ABORT18, S_ALTMODE1, S_BREAK1, S_CALL1, S_CLEAR_INPUT1, S_CLEAR_SCREEN1, S_DELETE1, S_END1, S_HELP1, S_HOLD_OUTPUT1, S_MACRO1, S_M_LOCK1, S_NETWORK1, S_OVER_STRIKE1, S_QUOTE_MOD1, S_RESUME1, S_RETURN1, S_STATUS1, S_STOP_OUTPUT1, S_SYSTEM1, S_TERMINAL1: footprint Button_Switch_Keyboard:SW_MX_2U -> Button_Switch_Keyboard:SW_Cherry_MX_2.00u_PCB
- S_BACKSLASH1, S_CTRL1, S_LEFT_ALT1, S_LGREEK1, S_LHYPER1, S_LMETA1, S_LSUPER1, S_LTOP1, S_RCTRL1, S_REPEAT1, S_RHYPER1, S_RIGHT_ALT1, S_RMETA1, S_RSUPER1, S_RTOP1, S_TAB1: footprint Button_Switch_Keyboard:SW_MX_1.5U -> Button_Switch_Keyboard:SW_Cherry_MX_1.50u_PCB
- S_EQ1: footprint Button_Switch_Keyboard:SW_MX_1.5U -> Button_Switch_Keyboard:SW_Cherry_MX_1.00u_PCB; dep S_MINUS1 -> S_PLUS1
- S_FN1: footprint Button_Switch_Keyboard:SW_MX_1U -> Button_Switch_Keyboard:SW_Cherry_MX_1.50u_PCB
- S_LINE1: footprint Button_Switch_Keyboard:SW_MX_1.25U -> Button_Switch_Keyboard:SW_Cherry_MX_1.25u_PCB
- S_LSHIFT1: footprint Button_Switch_Keyboard:SW_MX_2.25U -> Button_Switch_Keyboard:SW_Cherry_MX_2.25u_PCB
- S_MINUS1, S_RGREEK1: footprint Button_Switch_Keyboard:SW_MX_1.5U -> Button_Switch_Keyboard:SW_Cherry_MX_1.00u_PCB
- S_RIGHT_SPACE1: footprint Button_Switch_Keyboard:SW_MX_3U -> Button_Switch_Keyboard:SW_Cherry_MX_2.25u_PCB; dep S_LEFT_SPC17 -> S_LEFT_SPACE1
- S_RKM1: renamed from S_LKM1; value LKM -> RKM; footprint Button_Switch_Keyboard:SW_MX_1.25U -> Button_Switch_Keyboard:SW_Cherry_MX_1.25u_PCB; dep S_RIGHT_SPACE1 -> S_LKM1
- S_RSHIFT1: footprint Button_Switch_Keyboard:SW_MX_2.25U -> Button_Switch_Keyboard:SW_Cherry_MX_2.75u_PCB
- S_RUBOUT1: footprint Button_Switch_Keyboard:SW_MX_1.75U -> Button_Switch_Keyboard:SW_Cherry_MX_1.75u_PCB
Other:
- moved on the sheet: D_EQ1, D_LCURVEP1, D_RCURVEP1, D_STATUS1, D_THUMB_DOWN1, D_THUMB_UP1, S_EQ1, S_LCURVEP1, S_RCURVEP1, S_STATUS1, S_THUMB_DOWN1, S_THUMB_UP1

Commit message: wip: tkl-backspace
Parts:
- removed D_RCURVEP1: D, Diode_SMD:D_SOD-123, symbol Device:D_Small
- removed S_RCURVEP1: RCURVEP, Button_Switch_Keyboard:SW_Cherry_MX_1.00u_PCB, symbol Space_Cadet_Button_Switches:SWK
- S_BACKSPACE1: renamed from S_LCURVEP1; value LCURVEP -> BACKSPACE; footprint Button_Switch_Keyboard:SW_Cherry_MX_1.00u_PCB -> Button_Switch_Keyboard:SW_Cherry_MX_2.00u_PCB
- S_RIGHT_ALT1: dep S_LKM1 -> S_RKM1
- S_STATUS1: dep S_RCURVEP1 -> S_BACKSPACE1
- renumbered D_LCURVEP1 to D_BACKSPACE1
Other:
- moved on the sheet: D_THUMB_LEFT1, D_THUMB_RIGHT1, S_THUMB_LEFT1, S_THUMB_RIGHT1
Changed lines of the file:
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@@
 	(symbol
 		(lib_id "Device:D_Small")
-		(at 386.08 74.93 270)
-		(unit 1)
-		(exclude_from_sim no)
-		(in_bom yes)
-		(on_board yes)
-		(dnp no)
-		(fields_autoplaced yes)
-		(property "Reference" "D_RCURVEP1"
-			(at 388.62 73.6599 90)
-			(effects
-				(font
-					(size 1.27 1.27)
-				)
-				(justify left)
-			)
-		)
-		(property "Value" "D"
-			(at 388.62 76.1999 90)
-			(effects
-				(font
-					(size 1.27 1.27)
-				)
-				(justify left)
-			)
-		)
-		(property "Footprint" "Diode_SMD:D_SOD-123"
-			(at 386.08 74.93 90)
-			(effects
-				(font
-					(size 1.27 1.27)
-				)
-				(hide yes)
-			)
-		)
-		(property "Datasheet" "~"
-			(at 386.08 74.93 90)
-			(effects
-				(font
-					(size 1.27 1.27)
-				)
-				(hide yes)
-			)
-		)
-		(property "Description" "Diode, small symbol"
-			(at 386.08 74.93 0)
-			(effects
-				(font
-					(size 1.27 1.27)
-				)
-				(hide yes)
-			)
-		)
-		(property "Sim.Device" "D"
-			(at 386.08 74.93 0)
-			(effects
-				(font
-					(size 1.27 1.27)
-				)
-				(hide yes)
-			)
-		)
-		(property "Sim.Pins" "1=K 2=A"
-			(at 386.08 74.93 0)
-			(effects
-				(font
-					(size 1.27 1.27)
-				)
-				(hide yes)
-			)
-		)
-		(pin "1"
-		)
-		(pin "2"
-		)
-		(instances
-			(project "SpaceCadet"
-				(path "/4f7acbe2-a0f9-477a-99f4-186b01302303/1a8342a5-15fc-454c-84eb-2b470c08f569"
-					(reference "D_RCURVEP1")
-					(unit 1)
-				)
-			)
-		)
-	)
-	(symbol
-		(lib_id "Device:D_Small")
 		(at 214.63 74.93 270)
 		(unit 1)
@@
 	(symbol
 		(lib_id "Device:D_Small")
-		(at 424.18 95.25 270)
+		(at 443.23 95.25 270)
 		(unit 1)
 		(exclude_from_sim no)
@@
 		(dnp no)
 		(property "Reference" "D_THUMB_RIGHT1"
-			(at 426.212 93.98 90)
+			(at 445.262 93.98 90)
 			(effects
 				(font
@@
 		)
 		(property "Value" "D"
-			(at 426.72 96.5199 90)
+			(at 445.77 96.5199 90)
 			(effects
 				(font
@@
 		)
 		(property "Footprint" "Diode_SMD:D_SOD-123"
-			(at 424.18 95.25 90)
+			(at 443.23 95.25 90)
 			(effects
 				(font
@@
 		)
 		(property "Datasheet" "~"
-			(at 424.18 95.25 90)
+			(at 443.23 95.25 90)
 			(effects
 				(font
@@
 		)
 		(property "Description" "Diode, small symbol"
-			(at 424.18 95.25 0)
+			(at 443.23 95.25 0)
 			(effects
 				(font
@@
 		)
 		(property "Sim.Device" "D"
-			(at 424.18 95.25 0)
+			(at 443.23 95.25 0)
 			(effects
 				(font
@@
 		)
 		(property "Sim.Pins" "1=K 2=A"
-			(at 424.18 95.25 0)
+			(at 443.23 95.25 0)
 			(effects
 				(font
@@
 	(symbol
 		(lib_id "Space_Cadet_Button_Switches:SWK")
-		(at 415.036 105.41 0)
+		(at 434.086 105.41 0)
 		(unit 1)
 		(exclude_from_sim no)
@@
 		(dnp no)
 		(property "Reference" "S_THUMB_LEFT1"
-			(at 412.75 104.394 0)
+			(at 431.8 104.394 0)
 			(effects
 				(font
@@
 		)
 		(property "Value" "THUMB_LEFT"
-			(at 412.75 106.68 0)
+			(at 431.8 106.68 0)
 			(effects
 				(font
@@
 		)
 		(property "Footprint" "Button_Switch_Keyboard:SW_Cherry_MX_1.00u_PCB"
-			(at 415.544 107.95 0)
+			(at 434.594 107.95 0)
 			(effects
 				(font
@@
 		)
 		(property "Datasheet" ""
-			(at 424.434 106.934 0)
+			(at 443.484 106.934 0)
 			(effects
 				(font
@@
 		)
 		(property "Description" ""
-			(at 415.036 105.41 0)
+			(at 434.086 105.41 0)
 			(effects
 				(font
@@
 		)
 		(property "dep" "S_DELETE1"
-			(at 415.036 105.41 0)
+			(at 434.086 105.41 0)
 			(effects
 				(font
@@
 	(symbol
 		(lib_id "Space_Cadet_Button_Switches:SWK")
-		(at 394.97 85.09 0)
-		(unit 1)
-		(exclude_from_sim no)
-		(in_bom yes)
-		(on_board yes)
-		(dnp no)
-		(fields_autoplaced yes)
-		(property "Reference" "S_RCURVEP1"
-			(at 392.43 83.8199 0)
-			(effects
-				(font
-					(size 1.27 1.27)
-				)
-				(justify right)
-			)
-		)
-		(property "Value" "RCURVEP"
-			(at 392.43 86.3599 0)
-			(effects
-				(font
-					(size 1.27 1.27)
-				)
-				(justify right)
-			)
-		)
-		(property "Footprint" "Button_Switch_Keyboard:SW_Cherry_MX_1.00u_PCB"
-			(at 395.478 87.63 0)
-			(effects
-				(font
-					(size 1.27 1.27)
-				)
-				(hide yes)
-			)
-		)
-		(property "Datasheet" ""
-			(at 404.368 86.614 0)
-			(effects
-				(font
-					(size 1.27 1.27)
-				)
-				(hide yes)
-			)
-		)
-		(property "Description" ""
-			(at 394.97 85.09 0)
-			(effects
-				(font
-					(size 1.27 1.27)
-				)
-				(hide yes)
-			)
-		)
-		(property "dep" "S_LCURVEP1"
-			(at 394.97 85.09 0)
-			(effects
-				(font
-					(size 1.27 1.27)
-				)
-				(hide yes)
-			)
-		)
-		(pin "1"
-		)
-		(pin "2"
-		)
-		(instances
-			(project "SpaceCadet"
-				(path "/4f7acbe2-a0f9-477a-99f4-186b01302303/1a8342a5-15fc-454c-84eb-2b470c08f569"
-					(reference "S_RCURVEP1")
-					(unit 1)
-				)
-			)
-		)
-	)
-	(symbol
-		(lib_id "Space_Cadet_Button_Switches:SWK")
 		(at 318.516 105.41 0)
 		(unit 1)
@@
 	(symbol
 		(lib_id "Device:D_Small")
-		(at 405.13 95.25 270)
+		(at 424.18 95.25 270)
 		(unit 1)
 		(exclude_from_sim no)
@@
 		(dnp no)
 		(property "Reference" "D_THUMB_LEFT1"
-			(at 406.654 93.98 90)
+			(at 425.704 93.98 90)
 			(effects
 				(font
@@
 		)
 		(property "Value" "D"
-			(at 407.67 96.5199 90)
+			(at 426.72 96.5199 90)
 			(effects
 				(font
@@
 		)
 		(property "Footprint" "Diode_SMD:D_SOD-123"
-			(at 405.13 95.25 90)
+			(at 424.18 95.25 90)
 			(effects
 				(font
@@
 		)
 		(property "Datasheet" "~"
-			(at 405.13 95.25 90)
+			(at 424.18 95.25 90)
 			(effects
 				(font
@@
 		)
 		(property "Description" "Diode, small symbol"
-			(at 405.13 95.25 0)
+			(at 424.18 95.25 0)
 			(effects
 				(font
@@
 		)
 		(property "Sim.Device" "D"
-			(at 405.13 95.25 0)
+			(at 424.18 95.25 0)
 			(effects
 				(font
@@
 		)
 		(property "Sim.Pins" "1=K 2=A"
-			(at 405.13 95.25 0)
+			(at 424.18 95.25 0)
 			(effects
 				(font
@@
 		(dnp no)
 		(fields_autoplaced yes)
-		(property "Reference" "S_LCURVEP1"
+		(property "Reference" "S_BACKSPACE1"
 			(at 373.38 83.8199 0)
 			(effects
@@
 			)
 		)
-		(property "Value" "LCURVEP"
+		(property "Value" "BACKSPACE"
 			(at 373.38 86.3599 0)
 			(effects
@@
 			)
 		)
-		(property "Footprint" "Button_Switch_Keyboard:SW_Cherry_MX_1.00u_PCB"
+		(property "Footprint" "Button_Switch_Keyboard:SW_Cherry_MX_2.00u_PCB"
 			(at 376.428 87.63 0)
 			(effects
@@
 			(project "SpaceCadet"
 				(path "/4f7acbe2-a0f9-477a-99f4-186b01302303/1a8342a5-15fc-454c-84eb-2b470c08f569"
-					(reference "S_LCURVEP1")
+					(reference "S_BACKSPACE1")
 					(unit 1)
 				)
@@
 			)
 		)
-		(property "dep" "S_LKM1"
+		(property "dep" "S_RKM1"
 			(at 356.616 172.72 0)
 			(effects
@@
 	(symbol
 		(lib_id "Space_Cadet_Button_Switches:SWK")
-		(at 432.816 106.68 0)
+		(at 451.866 106.68 0)
 		(unit 1)
 		(exclude_from_sim no)
@@
 		(dnp no)
 		(property "Reference" "S_THUMB_RIGHT1"
-			(at 431.038 105.664 0)
+			(at 450.088 105.664 0)
 			(effects
 				(font
@@
 		)
 		(property "Value" "THUMB_RIGHT"
-			(at 431.038 107.95 0)
+			(at 450.088 107.95 0)
 			(effects
 				(font
@@
 		)
 		(property "Footprint" "Button_Switch_Keyboard:SW_Cherry_MX_1.00u_PCB"
-			(at 433.324 109.22 0)
+			(at 452.374 109.22 0)
 			(effects
 				(font
@@
 		)
 		(property "Datasheet" ""
-			(at 442.214 108.204 0)
+			(at 461.264 108.204 0)
 			(effects
 				(font
@@
 		)
 		(property "Description" ""
-			(at 432.816 106.68 0)
+			(at 451.866 106.68 0)
 			(effects
 				(font
@@
 		)
 		(property "dep" "S_THUMB_LEFT1"
-			(at 432.816 106.68 0)
+			(at 451.866 106.68 0)
 			(effects
 				(font
@@
 			)
 		)
-		(property "dep" "S_RCURVEP1"
+		(property "dep" "S_BACKSPACE1"
 			(at 413.766 85.09 0)
 			(effects
@@
 		(on_board yes)
 		(dnp no)
-		(fields_autoplaced yes)
-		(property "Reference" "D_LCURVEP1"
+		(property "Reference" "D_BACKSPACE1"
 			(at 369.57 73.6599 90)
 			(effects
@@
 			(project "SpaceCadet"
 				(path "/4f7acbe2-a0f9-477a-99f4-186b01302303/1a8342a5-15fc-454c-84eb-2b470c08f569"
-					(reference "D_LCURVEP1")
+					(reference "D_BACKSPACE1")
 					(unit 1)
 				)

Commit message: fix: right shift front, add img/layout.png
Parts:
- S_RGREEK1: footprint Button_Switch_Keyboard:SW_Cherry_MX_1.00u_PCB -> Button_Switch_Keyboard:SW_Cherry_MX_1.50u_Plate
- S_RSHIFT1: footprint Button_Switch_Keyboard:SW_Cherry_MX_2.75u_PCB -> Button_Switch_Keyboard:SW_Cherry_MX_2.25u_PCB
Changed lines of the file:
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@@
 			)
 		)
-		(property "Footprint" "Button_Switch_Keyboard:SW_Cherry_MX_1.00u_PCB"
+		(property "Footprint" "Button_Switch_Keyboard:SW_Cherry_MX_1.50u_Plate"
 			(at 338.074 153.67 0)
 			(effects
@@
 			)
 		)
-		(property "Footprint" "Button_Switch_Keyboard:SW_Cherry_MX_2.75u_PCB"
+		(property "Footprint" "Button_Switch_Keyboard:SW_Cherry_MX_2.25u_PCB"
 			(at 319.024 153.67 0)
 			(effects
