File: SpaceCadet.kicad_pcb (KiCad board)
At the start: 2 copper layers, 473.9 x 133 mm, 105 parts

Commit message: wip: pcb+hypo
Parts:
- removed S_LEFT_SPC17: LEFT_SPACE, Button_Switch_Keyboard:SW_MX_3U
- added S_LEFT_SPACE1: LEFT_SPACE, Button_Switch_Keyboard:SW_Cherry_MX_2.75u_PCB, F.Cu at (222.8, 123.5)
- added S_LHYPO1: LEFT_HYPO, Button_Switch_Keyboard:SW_Cherry_MX_6.25u_PCB, F.Cu at (84.6, 155.0)
- added S_PLUS1: PLUS, Button_Switch_Keyboard:SW_Cherry_MX_1.00u_PCB, F.Cu at (339.4, 47.3)
- added S_RHYPO1: RIGHT_HYPO, Button_Switch_Keyboard:SW_Cherry_MX_6.25u_PCB, F.Cu at (420.5, 155.0)
- added S_RKM1: RKM, Button_Switch_Keyboard:SW_Cherry_MX_1.25u_PCB, F.Cu at (327.5, 123.5)
- S_A1, S_ALTLOCK1, S_B1, S_BACKTICK1, S_C1, S_CAPSLOCK1, S_COLON1, S_COMMA1, S_D1, S_DOT1, S_E1, S_EIGHT1, S_F1, S_FIVE1, S_FOUR1, S_G1, S_H1, S_I_1, S_J1, S_K1, S_L1, S_LCURVEP1, S_LPAREN1, S_M17, S_N1, S_NINE1, S_O1, S_ONE1, S_P1, S_Q1, S_QUOTE1, S_R1, S_RCURVEP1, S_ROM_FOUR1, S_ROM_ONE1, S_ROM_THREE1, S_ROM_TWO1, S_RPAREN1, S_S1, S_SEMICOLON1, S_SEVEN1, S_SIX1, S_SLASH1, S_T1, S_THREE1, S_THUMB_DOWN1, S_THUMB_LEFT1, S_THUMB_RIGHT1, S_THUMB_UP1, S_TWO1, S_U1, S_V1, S_W1, S_X1, S_Y1, S_Z1, S_ZERO1: footprint Button_Switch_Keyboard:SW_MX_1U -> Button_Switch_Keyboard:SW_Cherry_MX_1.00u_PCB
- S_ABORT18, S_ALTMODE1, S_BREAK1, S_CALL1, S_CLEAR_INPUT1, S_CLEAR_SCREEN1, S_DELETE1, S_END1, S_HELP1, S_HOLD_OUTPUT1, S_MACRO1, S_M_LOCK1, S_NETWORK1, S_OVER_STRIKE1, S_QUOTE_MOD1, S_RESUME1, S_RETURN1, S_STATUS1, S_STOP_OUTPUT1, S_SYSTEM1, S_TERMINAL1: footprint Button_Switch_Keyboard:SW_MX_2U -> Button_Switch_Keyboard:SW_Cherry_MX_2.00u_PCB
- S_BACKSLASH1, S_CTRL1, S_LEFT_ALT1, S_LGREEK1, S_LHYPER1, S_LMETA1, S_LSUPER1, S_LTOP1, S_RCTRL1, S_REPEAT1, S_RHYPER1, S_RIGHT_ALT1, S_RMETA1, S_RSUPER1, S_RTOP1, S_TAB1: footprint Button_Switch_Keyboard:SW_MX_1.5U -> Button_Switch_Keyboard:SW_Cherry_MX_1.50u_PCB
- S_EQ1, S_MINUS1, S_RGREEK1: footprint Button_Switch_Keyboard:SW_MX_1.5U -> Button_Switch_Keyboard:SW_Cherry_MX_1.00u_PCB
- S_FN1: footprint Button_Switch_Keyboard:SW_MX_1U -> Button_Switch_Keyboard:SW_Cherry_MX_1.50u_PCB
- S_LINE1, S_LKM1: footprint Button_Switch_Keyboard:SW_MX_1.25U -> Button_Switch_Keyboard:SW_Cherry_MX_1.25u_PCB
- S_LSHIFT1: footprint Button_Switch_Keyboard:SW_MX_2.25U -> Button_Switch_Keyboard:SW_Cherry_MX_2.25u_PCB
- S_RIGHT_SPACE1: footprint Button_Switch_Keyboard:SW_MX_3U -> Button_Switch_Keyboard:SW_Cherry_MX_2.25u_PCB
- S_RSHIFT1: footprint Button_Switch_Keyboard:SW_MX_2.25U -> Button_Switch_Keyboard:SW_Cherry_MX_2.75u_PCB
- S_RUBOUT1: footprint Button_Switch_Keyboard:SW_MX_1.75U -> Button_Switch_Keyboard:SW_Cherry_MX_1.75u_PCB
- moved S_LKM1 25.7 mm to (303.7, 123.5)
- moved S_RIGHT_SPACE1 19.2 mm to (270.4, 123.5)
- moved S_MINUS1 10.2 mm to (320.4, 47.3)
- moved S_RGREEK1 9.88 mm to (396.6, 104.5)
- moved S_RSHIFT1 9.88 mm to (360.9, 104.5)
- moved S_FN1 9.88 mm to (182.3, 123.5)
- moved S_EQ1 9.88 mm to (358.5, 47.3)
- moved S_THUMB_DOWN1 8.86 mm to (472.8, 47.3)
- moved S_THUMB_RIGHT1 8.86 mm to (472.8, 66.4)
- moved S_THUMB_UP1 8.86 mm to (453.7, 47.3)
- moved S_RCURVEP1 8.86 mm to (396.6, 47.3)
- moved S_STATUS1 8.86 mm to (425.2, 47.3)
- moved S_LCURVEP1 8.86 mm to (377.5, 47.3)
- moved S_U1 8.86 mm to (253.7, 66.4)
- moved S_K1 8.86 mm to (277.5, 85.4)
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Other:
- board size 473.9 x 133 mm -> 473.9 x 164.9 mm

Commit message: wip: tkl-backspace
Parts:
- removed S_LCURVEP1: LCURVEP, Button_Switch_Keyboard:SW_Cherry_MX_1.00u_PCB
- removed S_RCURVEP1: RCURVEP, Button_Switch_Keyboard:SW_Cherry_MX_1.00u_PCB
- added S_BACKSPACE1: BACKSPACE, Button_Switch_Keyboard:SW_Cherry_MX_2.00u_PCB, F.Cu at (387.4, 48.9)
- moved S_RHYPO1 3.01 mm to (423.1, 156.6)
- moved S_QUOTE1 1.59 mm to (335.0, 87.0)
- moved S_ABORT18 1.59 mm to (349.3, 29.8)
- moved S_COMMA1 1.59 mm to (287.4, 106.0)
- moved S_HELP1 1.59 mm to (463.6, 87.0)
- moved S_J1 1.59 mm to (258.8, 87.0)
- moved S_K1 1.59 mm to (277.8, 87.0)
- moved S_LEFT_SPACE1 1.59 mm to (223.1, 125.1)
- moved S_RETURN1 1.59 mm to (363.6, 87.0)
- moved S_RGREEK1 1.59 mm to (396.9, 106.0)
- moved S_RIGHT_SPACE1 1.59 mm to (270.7, 125.1)
- moved S_RTOP1 1.59 mm to (420.7, 106.0)
- moved S_SLASH1 1.59 mm to (325.5, 106.0)
- moved S_RESUME1 1.59 mm to (425.5, 29.8)
- moved S_END1 1.59 mm to (425.5, 87.0)
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
Commit message: fix backspace
Parts:
- moved S_LHYPO1 55.3 mm to (139.8, 163.3)
- moved S_RHYPO1 35.8 mm to (388.0, 163.3)
- moved S_ALTLOCK1 5.18 mm to (478.0, 107.8)
- moved S_C1 5.18 mm to (197.0, 107.8)
- moved S_CAPSLOCK1 5.18 mm to (39.8, 107.8)
- moved S_COMMA1 5.18 mm to (292.2, 107.8)
- moved S_DOT1 5.18 mm to (311.3, 107.8)
- moved S_FN1 5.18 mm to (187.5, 126.8)
- moved S_LEFT_SPACE1 5.18 mm to (227.9, 126.8)
- moved S_LGREEK1 5.18 mm to (92.2, 107.8)
- moved S_LKM1 5.18 mm to (308.9, 126.8)
- moved S_LSHIFT1 5.18 mm to (127.9, 107.8)
- moved S_M17 5.18 mm to (273.2, 107.8)
- moved S_N1 5.18 mm to (254.1, 107.8)
- moved S_RCTRL1 5.18 mm to (387.5, 126.8)
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Other:
- board size 473.9 x 164.9 mm -> 485.5 x 184.6 mm

Commit message: fix: right shift front, add img/layout.png
Parts:
- S_RGREEK1: footprint Button_Switch_Keyboard:SW_Cherry_MX_1.00u_PCB -> Button_Switch_Keyboard:SW_Cherry_MX_1.50u_Plate
- S_RSHIFT1: footprint Button_Switch_Keyboard:SW_Cherry_MX_2.75u_PCB -> Button_Switch_Keyboard:SW_Cherry_MX_2.25u_PCB
- moved S_RHYPO1 9.97 mm to (378.1, 161.8)
- moved S_RGREEK1 7.17 mm to (394.8, 106.2)
- moved S_RSHIFT1 7.17 mm to (359.1, 106.2)
- moved S_LHYPO1 4.87 mm to (135.2, 161.8)
- moved S_RESUME1 2.73 mm to (428.1, 30.0)
- moved S_J1 2.73 mm to (261.4, 87.2)
- moved S_ABORT18 2.73 mm to (351.9, 30.0)
- moved S_M17 2.73 mm to (271.0, 106.2)
- moved S_RTOP1 2.73 mm to (423.4, 106.2)
- moved S_SLASH1 2.73 mm to (328.1, 106.2)
- moved S_HOLD_OUTPUT1 2.73 mm to (275.7, 30.0)
- moved S_QUOTE1 2.73 mm to (337.6, 87.2)
- moved S_K1 2.73 mm to (280.5, 87.2)
- moved S_SEMICOLON1 2.73 mm to (318.6, 87.2)
- moved S_ALTLOCK1 2.73 mm to (475.7, 106.2)
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
Commit message: fixes: bottom line and backspace, keyboard-layout.json added (keyboard-layout-editor.com)
Parts:
- removed S_BACKSPACE1: BACKSPACE, Button_Switch_Keyboard:SW_Cherry_MX_2.00u_PCB
- removed S_CTRL1: LEFT_CTRL, Button_Switch_Keyboard:SW_Cherry_MX_1.50u_PCB
- removed S_FN1: FN, Button_Switch_Keyboard:SW_Cherry_MX_1.50u_PCB
- removed S_LEFT_ALT1: LEFT_ALT, Button_Switch_Keyboard:SW_Cherry_MX_1.50u_PCB
- removed S_LEFT_SPACE1: LEFT_SPACE, Button_Switch_Keyboard:SW_Cherry_MX_2.75u_PCB
- removed S_LKM1: LKM, Button_Switch_Keyboard:SW_Cherry_MX_1.25u_PCB
- removed S_PLUS1: PLUS, Button_Switch_Keyboard:SW_Cherry_MX_1.00u_PCB
- removed S_RIGHT_ALT1: RIGHT_ALT, Button_Switch_Keyboard:SW_Cherry_MX_1.50u_PCB
- removed S_RIGHT_SPACE1: RIGHT_SPACE, Button_Switch_Keyboard:SW_Cherry_MX_2.25u_PCB
- removed S_RKM1: RKM, Button_Switch_Keyboard:SW_Cherry_MX_1.25u_PCB
- added S_LBACK1: LBACK, Button_Switch_Keyboard:SW_Cherry_MX_1.25u_PCB, F.Cu at (159.9, 126.6)
- added S_LBOTTOM1: LEFT_BOTTOM, Button_Switch_Keyboard:SW_Cherry_MX_1.25u_PCB, F.Cu at (183.7, 126.6)
- added S_LCTRL1: LEFT_CTRL, Button_Switch_Keyboard:SW_Cherry_MX_1.75u_PCB, F.Cu at (131.3, 126.6)
- added S_LCURVE1: LEFT_CURVE, Button_Switch_Keyboard:SW_Cherry_MX_1.00u_PCB, F.Cu at (381.4, 50.4)
- added S_LSPACE1: LEFT_SPACE, Button_Switch_Keyboard:SW_Cherry_MX_2.75u_PCB, F.Cu at (221.8, 126.6)
- added S_RBACK1: RIGHT_BACK, Button_Switch_Keyboard:SW_Cherry_MX_1.25u_PCB, F.Cu at (326.6, 126.6)
- added S_RBOTTOM1: RIGHT_BOTTOM, Button_Switch_Keyboard:SW_Cherry_MX_1.25u_PCB, F.Cu at (302.8, 126.6)
- added S_RCURVE1: RIGHT_CURVE, Button_Switch_Keyboard:SW_Cherry_MX_1.00u_PCB, F.Cu at (400.4, 50.4)
- added S_RFN1: RIGHT_FN, Button_Switch_Keyboard:SW_Cherry_MX_1.50u_PCB, F.Cu at (386.1, 126.6)
- added S_RSPACE1: RIGHT_SPACE, Button_Switch_Keyboard:SW_Cherry_MX_2.25u_PCB, F.Cu at (269.5, 126.6)
- S_EQ1: value EQ -> EQUAL; footprint Button_Switch_Keyboard:SW_Cherry_MX_1.00u_PCB -> Button_Switch_Keyboard:SW_Cherry_MX_1.50u_PCB
- S_MINUS1: footprint Button_Switch_Keyboard:SW_Cherry_MX_1.00u_PCB -> Button_Switch_Keyboard:SW_Cherry_MX_1.50u_PCB
- S_RCTRL1: footprint Button_Switch_Keyboard:SW_Cherry_MX_1.50u_PCB -> Button_Switch_Keyboard:SW_Cherry_MX_1.75u_PCB
- moved S_RCTRL1 30.1 mm to (355.2, 126.6)
- moved S_MINUS1 5.79 mm to (329.0, 50.4)
- moved S_EQ1 4.09 mm to (357.6, 50.4)
- moved S_STATUS1 1.57 mm to (429.0, 50.4)
- moved S_THUMB_UP1 1.57 mm to (457.6, 50.4)
- moved S_THUMB_DOWN1 1.57 mm to (476.6, 50.4)
- moved S_RESUME1 1.57 mm to (429.0, 31.3)
- moved S_ALTLOCK1 1.57 mm to (476.6, 107.5)
- moved S_DOT1 1.57 mm to (309.9, 107.5)
- moved S_J1 1.57 mm to (262.3, 88.5)
- moved S_LPAREN1 1.57 mm to (333.7, 69.4)
- moved S_M17 1.57 mm to (271.8, 107.5)
- moved S_NINE1 1.57 mm to (286.1, 50.4)
- moved S_O1 1.57 mm to (295.6, 69.4)
- moved S_REPEAT1 1.57 mm to (452.8, 107.5)
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
Commit message: wip: display2004 added, fixed to original SpaceCadet layout
Parts:
- added DISPLAY1: LCD-20X4, Button_Switch_Keyboard:lcd-2004, F.Cu at (254.5, 172.6)
- moved S_LHYPO1 9.97 mm to (126.2, 163.7)
- moved S_RHYPO1 9.16 mm to (388.1, 163.7)
- moved S_HELP1 1.06 mm to (466.7, 87.5)
- moved S_LINE1 1.06 mm to (397.6, 87.5)
- moved S_QUOTE1 1.06 mm to (338.1, 87.5)
- moved S_SEMICOLON1 1.06 mm to (319.1, 87.5)
- moved S_A1 1.06 mm to (147.6, 87.5)
- moved S_ALTMODE1 1.06 mm to (85.7, 87.5)
- moved S_G1 1.06 mm to (223.8, 87.5)
- moved S_H1 1.06 mm to (242.9, 87.5)
- moved S_RUBOUT1 1.06 mm to (121.4, 87.5)
- moved S_S1 1.06 mm to (166.7, 87.5)
- moved S_L1 1.06 mm to (300.0, 87.5)
- moved S_RETURN1 1.06 mm to (366.7, 87.5)
- moved S_EIGHT1 1.06 mm to (266.7, 49.4)
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Other:
- board size 485.5 x 184.6 mm -> 485.5 x 200 mm
