File: SpaceCadet.kicad_pcb (KiCad board)
At the start: 2 copper layers, 473.2 x 186 mm, 220 parts, among them U101 Pico

Commit message: wip:wiring_5
Connections:
- D_LBOTTOM1 pad 1: COL7 -> ROW11
- D_LCTRL1 pad 1: COL7 -> ROW11
- D_LHYPO1 pad 1: COL7 -> ROW11
- D_LHYPO2 pad 1: COL7 -> ROW10
- D_LSUPER1 pad 1: COL7 -> ROW11
- D_RFN1 pad 1: COL7 -> ROW11
- D_RHYPO1 pad 1: COL7 -> ROW11
- D_RHYPO2 pad 1: COL7 -> ROW10
- S_LHYPO1 pad 3: Net-(D_LHYPO2-A) -> COL6
- S_LHYPO1 pad 4: COL7 -> Net-(D_LHYPO2-A)
- S_RHYPO1 pad 1: unconnected-(S_RHYPO1-in-Pad1) -> COL7
- S_RHYPO1 pad 3: Net-(D_RHYPO2-A) -> COL7
- S_RHYPO1 pad 4: unconnected-(S_RHYPO1-in-Pad4) -> Net-(D_RHYPO2-A)
Routing:
- net ROW11: track 0.00 -> 796.1 mm
- net (no net): track 619.1 -> 0.10 mm
- net ROW10: track 473.1 -> 815.7 mm, vias 0 -> 2
- net COL7: track 296.0 -> 433.7 mm
- net COL6: track 257.1 -> 365.0 mm
- net Net-(D_LHYPO2-A): track 0.00 -> 13.5 mm

Commit message: wip: schematic refactor
Connections:
- D_ABORT1 pad 1: ROW1 -> unconnected-(D_ABORT1-K-Pad1)
- D_ABORT1 pad 2: Net-(D_ABORT1-A) -> unconnected-(D_ABORT1-A-Pad2)
- D_ALTLOCK1 pad 2: Net-(D_ALTLOCK1-A) -> unconnected-(D_ALTLOCK1-A-Pad2)
- D_BACK1 pad 2: Net-(D_BACK1-A) -> unconnected-(D_BACK1-A-Pad2)
- D_BACKSLASH1 pad 2: Net-(D_BACKSLASH1-A) -> unconnected-(D_BACKSLASH1-A-Pad2)
- D_BACKTICK1 pad 2: Net-(D_BACKTICK1-A) -> unconnected-(D_BACKTICK1-A-Pad2)
- D_BREAK1 pad 1: ROW1 -> unconnected-(D_BREAK1-K-Pad1)
- D_BREAK1 pad 2: Net-(D_BREAK1-A) -> unconnected-(D_BREAK1-A-Pad2)
- D_CALL1 pad 1: ROW1 -> unconnected-(D_CALL1-K-Pad1)
- D_CALL1 pad 2: Net-(D_CALL1-A) -> unconnected-(D_CALL1-A-Pad2)
- D_CAPS_LOCK1 pad 2: Net-(D_CAPS_LOCK1-A) -> unconnected-(D_CAPS_LOCK1-A-Pad2)
- D_COLON1 pad 1: ROW3 -> ROW1
- D_COMMA1 pad 2: Net-(D_COMMA1-A) -> unconnected-(D_COMMA1-A-Pad2)
- D_D1 pad 2: Net-(D_D1-A) -> unconnected-(D_D1-A-Pad2)
- D_DELETE1 pad 2: Net-(D_DELETE1-A) -> unconnected-(D_DELETE1-A-Pad2)
- D_DOT1 pad 2: Net-(D_DOT1-A) -> unconnected-(D_DOT1-A-Pad2)
- D_EIGHT1 pad 1: ROW3 -> ROW1
- D_END1 pad 2: Net-(D_END1-A) -> unconnected-(D_END1-A-Pad2)
- D_EQ1 pad 1: ROW3 -> Net-(D_EQ1-K)
- D_EQ1 pad 2: Net-(D_EQ1-A) -> unconnected-(D_EQ1-A-Pad2)
- D_F1 pad 2: Net-(D_F1-A) -> unconnected-(D_F1-A-Pad2)
- D_FIVE1 pad 1: ROW2 -> ROW1
- D_FOUR1 pad 1: ROW3 -> ROW1
- D_G1 pad 2: Net-(D_G1-A) -> unconnected-(D_G1-A-Pad2)
- D_H1 pad 2: Net-(D_H1-A) -> unconnected-(D_H1-A-Pad2)
- D_HELP1 pad 2: Net-(D_HELP1-A) -> unconnected-(D_HELP1-A-Pad2)
- D_HOLD_OUTPUT1 pad 1: ROW1 -> unconnected-(D_HOLD_OUTPUT1-K-Pad1)
- D_HOLD_OUTPUT1 pad 2: Net-(D_HOLD_OUTPUT1-A) -> unconnected-(D_HOLD_OUTPUT1-A-Pad2)
- D_I_1 pad 2: Net-(D_I_1-A) -> unconnected-(D_I_1-A-Pad2)
- D_J1 pad 2: Net-(D_J1-A) -> unconnected-(D_J1-A-Pad2)
- D_K1 pad 2: Net-(D_K1-A) -> unconnected-(D_K1-A-Pad2)
- D_L1 pad 2: Net-(D_L1-A) -> unconnected-(D_L1-A-Pad2)
- D_LCTRL1 pad 2: Net-(D_LCTRL1-A) -> unconnected-(D_LCTRL1-A-Pad2)
- D_LCURVE1 pad 1: ROW2 -> Net-(D_LCURVE1-K)
- D_LCURVE1 pad 2: Net-(D_LCURVE1-A) -> unconnected-(D_LCURVE1-A-Pad2)
- D_LINE1 pad 2: Net-(D_LINE1-A) -> unconnected-(D_LINE1-A-Pad2)
- D_LPAREN1 pad 2: Net-(D_LPAREN1-A) -> unconnected-(D_LPAREN1-A-Pad2)
- D_LSPACE1 pad 2: Net-(D_LSPACE1-A) -> unconnected-(D_LSPACE1-A-Pad2)
- D_M1 pad 2: Net-(D_M1-A) -> unconnected-(D_M1-A-Pad2)
- D_MINUS1 pad 1: ROW2 -> Net-(D_LCURVE1-K)
- D_MINUS1 pad 2: Net-(D_MINUS1-A) -> unconnected-(D_MINUS1-A-Pad2)
- D_N1 pad 2: Net-(D_N1-A) -> unconnected-(D_N1-A-Pad2)
- D_NETWORK1 pad 2: Net-(D_NETWORK1-A) -> unconnected-(D_NETWORK1-A-Pad2)
- D_NINE1 pad 1: ROW2 -> Net-(D_LCURVE1-K)
- D_NINE1 pad 2: Net-(D_NINE1-A) -> unconnected-(D_NINE1-A-Pad2)
- D_O1 pad 2: Net-(D_O1-A) -> unconnected-(D_O1-A-Pad2)
- D_ONE1 pad 1: ROW2 -> ROW1
- D_P1 pad 2: Net-(D_P1-A) -> unconnected-(D_P1-A-Pad2)
- D_QUOTE1 pad 2: Net-(D_QUOTE1-A) -> unconnected-(D_QUOTE1-A-Pad2)
- D_R1 pad 2: Net-(D_R1-A) -> unconnected-(D_R1-A-Pad2)
- D_RBOTTOM1 pad 2: Net-(D_RBOTTOM1-A) -> unconnected-(D_RBOTTOM1-A-Pad2)
- D_RCTRL1 pad 2: Net-(D_RCTRL1-A) -> unconnected-(D_RCTRL1-A-Pad2)
- D_RCURVE1 pad 1: ROW3 -> Net-(D_EQ1-K)
- D_RCURVE1 pad 2: Net-(D_RCURVE1-A) -> unconnected-(D_RCURVE1-A-Pad2)
- D_REPEAT1 pad 2: Net-(D_REPEAT1-A) -> unconnected-(D_REPEAT1-A-Pad2)
- D_RESUME1 pad 1: ROW1 -> unconnected-(D_RESUME1-K-Pad1)
- D_RESUME1 pad 2: Net-(D_RESUME1-A) -> unconnected-(D_RESUME1-A-Pad2)
- D_RETURN1 pad 2: Net-(D_RETURN1-A) -> unconnected-(D_RETURN1-A-Pad2)
- D_RFN1 pad 2: Net-(D_RFN1-A) -> unconnected-(D_RFN1-A-Pad2)
- D_RGREEK1 pad 2: Net-(D_RGREEK1-A) -> unconnected-(D_RGREEK1-A-Pad2)
- D_RHYPER1 pad 2: Net-(D_RHYPER1-A) -> unconnected-(D_RHYPER1-A-Pad2)
- D_RMETA1 pad 2: Net-(D_RMETA1-A) -> unconnected-(D_RMETA1-A-Pad2)
- D_ROM_FOUR1 pad 2: Net-(D_ROM_FOUR1-A) -> unconnected-(D_ROM_FOUR1-A-Pad2)
- D_ROM_ONE1 pad 1: ROW2 -> ROW1
- D_ROM_THREE1 pad 2: Net-(D_ROM_THREE1-A) -> unconnected-(D_ROM_THREE1-A-Pad2)
- D_ROM_TWO1 pad 1: ROW3 -> ROW1
- D_RPAREN1 pad 2: Net-(D_RPAREN1-A) -> unconnected-(D_RPAREN1-A-Pad2)
- D_RSHIFT1 pad 2: Net-(D_RSHIFT1-A) -> unconnected-(D_RSHIFT1-A-Pad2)
- D_RSPACE1 pad 2: Net-(D_RSPACE1-A) -> unconnected-(D_RSPACE1-A-Pad2)
- D_RSUPER1 pad 2: Net-(D_RSUPER1-A) -> unconnected-(D_RSUPER1-A-Pad2)
- D_RTOP1 pad 2: Net-(D_RTOP1-A) -> unconnected-(D_RTOP1-A-Pad2)
- D_S1 pad 2: Net-(D_S1-A) -> unconnected-(D_S1-A-Pad2)
- D_SEMICOLON1 pad 2: Net-(D_SEMICOLON1-A) -> unconnected-(D_SEMICOLON1-A-Pad2)
- D_SEVEN1 pad 1: ROW2 -> ROW1
- D_SIX1 pad 1: ROW3 -> ROW1
- D_SLASH1 pad 2: Net-(D_SLASH1-A) -> unconnected-(D_SLASH1-A-Pad2)
- D_STATUS1 pad 1: ROW2 -> Net-(D_LCURVE1-K)
- D_STATUS1 pad 2: Net-(D_STATUS1-A) -> unconnected-(D_STATUS1-A-Pad2)
- D_STOP_OUTPUT1 pad 1: ROW1 -> unconnected-(D_STOP_OUTPUT1-K-Pad1)
- D_STOP_OUTPUT1 pad 2: Net-(D_STOP_OUTPUT1-A) -> unconnected-(D_STOP_OUTPUT1-A-Pad2)
- D_SYSTEM1 pad 1: ROW2 -> ROW1
- D_T1 pad 2: Net-(D_T1-A) -> unconnected-(D_T1-A-Pad2)
- D_THREE1 pad 1: ROW2 -> ROW1
- D_THUMB_DOWN1 pad 1: ROW2 -> Net-(D_LCURVE1-K)
- D_THUMB_DOWN1 pad 2: Net-(D_THUMB_DOWN1-A) -> unconnected-(D_THUMB_DOWN1-A-Pad2)
- D_THUMB_LEFT1 pad 2: Net-(D_THUMB_LEFT1-A) -> unconnected-(D_THUMB_LEFT1-A-Pad2)
- D_THUMB_RIGHT1 pad 2: Net-(D_THUMB_RIGHT1-A) -> unconnected-(D_THUMB_RIGHT1-A-Pad2)
- D_THUMB_UP1 pad 1: ROW3 -> Net-(D_EQ1-K)
- D_THUMB_UP1 pad 2: Net-(D_THUMB_UP1-A) -> unconnected-(D_THUMB_UP1-A-Pad2)
- D_TWO1 pad 1: ROW3 -> ROW1
- D_U1 pad 2: Net-(D_U1-A) -> unconnected-(D_U1-A-Pad2)
- D_X1 pad 2: Net-(D_X1-A) -> unconnected-(D_X1-A-Pad2)
- D_Y1 pad 2: Net-(D_Y1-A) -> unconnected-(D_Y1-A-Pad2)
- D_ZERO1 pad 1: ROW3 -> Net-(D_EQ1-K)
- D_ZERO1 pad 2: Net-(D_ZERO1-A) -> unconnected-(D_ZERO1-A-Pad2)
Routing:
- net ROW3: track 604.8 -> 0.00 mm
- net ROW2: track 498.5 -> 0.00 mm
- net Net-(D_EQ1-K): track 0.00 -> 261.0 mm
- net COL7: track 433.7 -> 392.7 mm
- net ROW1: track 447.9 -> 477.4 mm
- net unconnected-(D_HOLD_OUTPUT1-K-Pad1): track 0.00 -> 2.54 mm
- net unconnected-(D_ABORT1-K-Pad1): track 0.00 -> 2.54 mm
- net unconnected-(D_BREAK1-K-Pad1): track 0.00 -> 2.29 mm
- net unconnected-(D_STOP_OUTPUT1-K-Pad1): track 0.00 -> 2.26 mm
- net unconnected-(D_RESUME1-K-Pad1): track 0.00 -> 2.26 mm
- net unconnected-(D_CALL1-K-Pad1): track 0.00 -> 2.03 mm

Commit message: wip: unsplit & rewiring
Parts:
- removed D_LHYPO1, D_LHYPO2, D_RHYPO1, D_RHYPO2: D, Diode_THT:D_DO-41_SOD81_P7.62mm_Horizontal
- removed S_LHYPO1: LEFT_HYPO, Button_Switch_Keyboard:SW_Cherry_MX_6.25u_PCB
- removed S_RHYPO1: RIGHT_HYPO, Button_Switch_Keyboard:SW_Cherry_MX_6.25u_PCB
- S_A1, S_ALTLOCK1, S_B1, S_BACKTICK1, S_C1, S_CAPSLOCK1, S_COLON1, S_COMMA1, S_D1, S_DOT1, S_E1, S_EIGHT1, S_F1, S_FIVE1, S_FOUR1, S_G1, S_H1, S_I_1, S_J1, S_K1, S_L1, S_LCURVE1, S_LPAREN1, S_M1, S_N1, S_NINE1, S_O1, S_ONE1, S_P1, S_Q1, S_R1, S_RCURVE1, S_ROM_FOUR1, S_ROM_ONE1, S_ROM_THREE1, S_ROM_TWO1, S_RPAREN1, S_S1, S_SEMICOLON1, S_SEVEN1, S_SIX1, S_SLASH1, S_T1, S_THREE1, S_THUMB_DOWN1, S_THUMB_LEFT1, S_THUMB_RIGHT1, S_THUMB_UP1, S_TWO1, S_U1, S_V1, S_W1, S_X1, S_Y1, S_Z1, S_ZERO1: footprint Button_Switch_Keyboard:SW_Cherry_MX_1.00u_PCB -> Button_Switch_Keyboard:SWMXK_1.00u
- S_ABORT18, S_ALTMODE1, S_BREAK1, S_CALL1, S_CLEAR_INPUT1, S_CLEAR_SCREEN1, S_DELETE1, S_HELP1, S_HOLD_OUTPUT1, S_MACRO1, S_M_LOCK1, S_NETWORK1, S_OVER_STRIKE1, S_QUOTE_MOD1, S_RESUME1, S_RETURN1, S_STATUS1, S_STOP_OUTPUT1, S_SYSTEM1, S_TERMINAL1: footprint Button_Switch_Keyboard:SW_Cherry_MX_2.00u_PCB -> Button_Switch_Keyboard:SWMXK_2.00u
- S_BACKSLASH1, S_EQ1, S_MINUS1, S_REPEAT1, S_RFN1: footprint Button_Switch_Keyboard:SW_Cherry_MX_1.50u_PCB -> Button_Switch_Keyboard:SWMXK_1.00u
- S_END1: footprint Button_Switch_Keyboard:SW_Cherry_MX_2.00u_PCB -> Button_Switch_Keyboard:SWMXK_1.00u
- S_LBACK1, S_LBOTTOM1: footprint Button_Switch_Keyboard:SW_Cherry_MX_1.25u_PCB -> Button_Switch_Keyboard:SWMXK_1.25u
- S_LCTRL1, S_RUBOUT1: footprint Button_Switch_Keyboard:SW_Cherry_MX_1.75u_PCB -> Button_Switch_Keyboard:SWMXK_1.75u
- S_LGREEK1, S_LHYPER1, S_LMETA1, S_LSUPER1, S_LTOP1, S_RGREEK1, S_RHYPER1, S_RMETA1, S_RSUPER1, S_RTOP1: footprint Button_Switch_Keyboard:SW_Cherry_MX_1.50u_PCB -> Button_Switch_Keyboard:SWMXK_1.50u
- S_LINE1, S_RBACK1, S_RBOTTOM1: footprint Button_Switch_Keyboard:SW_Cherry_MX_1.25u_PCB -> Button_Switch_Keyboard:SWMXK_1.00u
- S_LSHIFT1: footprint Button_Switch_Keyboard:SW_Cherry_MX_2.25u_PCB -> Button_Switch_Keyboard:SWMXK_2.25u
- S_LSPACE1: footprint Button_Switch_Keyboard:SW_Cherry_MX_2.75u_PCB -> Button_Switch_Keyboard:SWMXK_1.00u
- S_QUOTE1: footprint Button_Switch_Keyboard:SW_Cherry_MX_1.00u_PCB -> Button_Switch_Keyboard:SWMXK_2.00u
- S_RCTRL1: footprint Button_Switch_Keyboard:SW_Cherry_MX_1.75u_PCB -> Button_Switch_Keyboard:SWMXK_1.00u
- S_RSHIFT1: footprint Button_Switch_Keyboard:SW_Cherry_MX_2.25u_PCB -> Button_Switch_Keyboard:SWMXK_1.50u
- S_RSPACE1: footprint Button_Switch_Keyboard:SW_Cherry_MX_2.25u_PCB -> Button_Switch_Keyboard:SWMXK_1.00u
- S_TAB1: footprint Button_Switch_Keyboard:SW_Cherry_MX_1.50u_PCB -> Button_Switch_Keyboard:SWMXK_1.75u
- moved D_LSHIFT1 3.08 mm to (118.4, 95.5)
- moved D_RUBOUT1 2.37 mm to (104.2, 76.5)
- moved D_LGREEK1 2.28 mm to (73.2, 95.5)
- moved D_OVER_STRIKE1 2.27 mm to (144.7, 19.4)
- moved D_CLEAR_INPUT1 2.24 mm to (182.8, 19.4)
- moved D_HOLD_OUTPUT1 2.24 mm to (259.0, 19.4)
- moved D_CLEAR_SCREEN1 2.24 mm to (220.9, 19.4)
- moved D_ABORT1 2.24 mm to (335.1, 19.4)
- moved D_LSUPER1 2.19 mm to (54.2, 114.6)
- moved D_CAPS_LOCK1 2.18 mm to (20.8, 95.5)
- moved D_TERMINAL1 2.16 mm to (68.4, 19.4)
- moved D_QUOTE_MOD1 2.16 mm to (106.6, 19.4)
- moved D_SYSTEM1 2.13 mm to (68.4, 38.4)
- moved D_LMETA1 2.12 mm to (82.7, 114.6)
- moved D_NETWORK1 2.10 mm to (68.4, 57.5)
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Connections:
- D_A1 pad 1: ROW7 -> ROW3
- D_ABORT1 pad 1: unconnected-(D_ABORT1-K-Pad1) -> ROW1
- D_ABORT1 pad 2: unconnected-(D_ABORT1-A-Pad2) -> Net-(D_ABORT1-A)
- D_ALTLOCK1 pad 1: ROW8 -> ROW4
- D_ALTLOCK1 pad 2: unconnected-(D_ALTLOCK1-A-Pad2) -> Net-(D_ALTLOCK1-A)
- D_ALTMODE1 pad 1: ROW7 -> ROW3
- D_B1 pad 1: ROW8 -> ROW4
- D_BACK1 pad 1: unconnected-(D_BACK1-K-Pad1) -> ROW6
- D_BACK1 pad 2: unconnected-(D_BACK1-A-Pad2) -> Net-(D_BACK1-A)
- D_BACKSLASH1 pad 1: ROW5 -> ROW8
- D_BACKSLASH1 pad 2: unconnected-(D_BACKSLASH1-A-Pad2) -> Net-(D_BACKSLASH1-A)
- D_BACKTICK1 pad 1: ROW4 -> ROW2
- D_BACKTICK1 pad 2: unconnected-(D_BACKTICK1-A-Pad2) -> Net-(D_BACKTICK1-A)
- D_BREAK1 pad 1: unconnected-(D_BREAK1-K-Pad1) -> ROW1
- D_BREAK1 pad 2: unconnected-(D_BREAK1-A-Pad2) -> Net-(D_BREAK1-A)
- D_C1 pad 1: ROW8 -> ROW4
- D_CALL1 pad 1: unconnected-(D_CALL1-K-Pad1) -> ROW2
- D_CALL1 pad 2: unconnected-(D_CALL1-A-Pad2) -> Net-(D_CALL1-A)
- D_CAPS_LOCK1 pad 1: ROW8 -> ROW4
- D_CAPS_LOCK1 pad 2: unconnected-(D_CAPS_LOCK1-A-Pad2) -> Net-(D_CAPS_LOCK1-A)
- D_COLON1 pad 1: ROW1 -> ROW2
- D_COMMA1 pad 1: ROW9 -> ROW6
- D_COMMA1 pad 2: unconnected-(D_COMMA1-A-Pad2) -> Net-(D_COMMA1-A)
- D_D1 pad 1: ROW7 -> ROW3
- D_D1 pad 2: unconnected-(D_D1-A-Pad2) -> Net-(D_D1-A)
- D_DELETE1 pad 1: ROW4 -> ROW2
- D_DELETE1 pad 2: unconnected-(D_DELETE1-A-Pad2) -> Net-(D_DELETE1-A)
- D_DOT1 pad 1: ROW8 -> ROW4
- D_DOT1 pad 2: unconnected-(D_DOT1-A-Pad2) -> Net-(D_DOT1-A)
- D_E1 pad 1: ROW4 -> ROW2
- D_EIGHT1 pad 1: ROW1 -> ROW2
- D_END1 pad 1: ROW7 -> ROW3
- D_END1 pad 2: unconnected-(D_END1-A-Pad2) -> Net-(D_END1-A)
- D_EQ1 pad 1: Net-(D_EQ1-K) -> ROW2
- D_EQ1 pad 2: unconnected-(D_EQ1-A-Pad2) -> Net-(D_EQ1-A)
- D_F1 pad 1: ROW6 -> ROW7
- D_F1 pad 2: unconnected-(D_F1-A-Pad2) -> Net-(D_F1-A)
- D_FIVE1 pad 1: ROW1 -> ROW10
- D_FOUR1 pad 1: ROW1 -> ROW2
- D_G1 pad 1: ROW7 -> ROW3
- D_G1 pad 2: unconnected-(D_G1-A-Pad2) -> Net-(D_G1-A)
- D_H1 pad 1: ROW6 -> ROW7
- D_H1 pad 2: unconnected-(D_H1-A-Pad2) -> Net-(D_H1-A)
- D_HELP1 pad 1: ROW6 -> ROW3
- D_HELP1 pad 2: unconnected-(D_HELP1-A-Pad2) -> Net-(D_HELP1-A)
- D_HOLD_OUTPUT1 pad 1: unconnected-(D_HOLD_OUTPUT1-K-Pad1) -> ROW1
- D_HOLD_OUTPUT1 pad 2: unconnected-(D_HOLD_OUTPUT1-A-Pad2) -> Net-(D_HOLD_OUTPUT1-A)
- D_I_1 pad 1: ROW5 -> ROW8
- D_I_1 pad 2: unconnected-(D_I_1-A-Pad2) -> Net-(D_I_1-A)
- D_J1 pad 1: ROW7 -> ROW3
- D_J1 pad 2: unconnected-(D_J1-A-Pad2) -> Net-(D_J1-A)
- D_K1 pad 2: unconnected-(D_K1-A-Pad2) -> Net-(D_K1-A)
- D_L1 pad 1: ROW6 -> ROW3
- D_L1 pad 2: unconnected-(D_L1-A-Pad2) -> Net-(D_L1-A)
- D_LBACK1 pad 1: ROW10 -> ROW5
- D_LBOTTOM1 pad 1: ROW11 -> ROW5
- D_LCTRL1 pad 1: ROW11 -> ROW5
- D_LCTRL1 pad 2: unconnected-(D_LCTRL1-A-Pad2) -> Net-(D_LCTRL1-A)
- D_LCURVE1 pad 1: Net-(D_LCURVE1-K) -> ROW10
- D_LCURVE1 pad 2: unconnected-(D_LCURVE1-A-Pad2) -> Net-(D_LCURVE1-A)
- D_LGREEK1 pad 1: ROW8 -> ROW4
- D_LHYPER1 pad 1: ROW10 -> ROW5
- D_LINE1 pad 1: ROW6 -> ROW3
- D_LINE1 pad 2: unconnected-(D_LINE1-A-Pad2) -> Net-(D_LINE1-A)
- D_LMETA1 pad 1: ROW10 -> ROW5
- D_LPAREN1 pad 1: ROW4 -> ROW2
- D_LPAREN1 pad 2: unconnected-(D_LPAREN1-A-Pad2) -> Net-(D_LPAREN1-A)
- D_LSHIFT1 pad 1: ROW9 -> ROW6
- D_LSPACE1 pad 1: ROW10 -> ROW5
- D_LSPACE1 pad 2: unconnected-(D_LSPACE1-A-Pad2) -> Net-(D_LSPACE1-A)
- D_LSUPER1 pad 1: ROW11 -> ROW6
- D_LTOP1 pad 1: ROW9 -> ROW7
- D_M1 pad 1: ROW8 -> ROW4
- D_M1 pad 2: unconnected-(D_M1-A-Pad2) -> Net-(D_M1-A)
- D_MINUS1 pad 1: Net-(D_LCURVE1-K) -> ROW10
- D_MINUS1 pad 2: unconnected-(D_MINUS1-A-Pad2) -> Net-(D_MINUS1-A)
- D_MODE_LOCK1 pad 1: ROW6 -> ROW3
- D_N1 pad 1: ROW9 -> ROW6
- D_N1 pad 2: unconnected-(D_N1-A-Pad2) -> Net-(D_N1-A)
- D_NETWORK1 pad 1: ROW4 -> ROW2
- D_NETWORK1 pad 2: unconnected-(D_NETWORK1-A-Pad2) -> Net-(D_NETWORK1-A)
- D_NINE1 pad 1: Net-(D_LCURVE1-K) -> ROW10
- D_NINE1 pad 2: unconnected-(D_NINE1-A-Pad2) -> Net-(D_NINE1-A)
- D_O1 pad 1: ROW4 -> ROW2
- D_O1 pad 2: unconnected-(D_O1-A-Pad2) -> Net-(D_O1-A)
- D_ONE1 pad 1: ROW1 -> ROW10
- D_P1 pad 1: ROW5 -> ROW8
- D_P1 pad 2: unconnected-(D_P1-A-Pad2) -> Net-(D_P1-A)
- D_Q1 pad 1: ROW4 -> ROW2
- D_QUOTE1 pad 1: ROW6 -> ROW3
- D_QUOTE1 pad 2: unconnected-(D_QUOTE1-A-Pad2) -> Net-(D_QUOTE1-A)
- D_R1 pad 1: ROW5 -> ROW8
- D_R1 pad 2: unconnected-(D_R1-A-Pad2) -> Net-(D_R1-A)
- D_RBOTTOM1 pad 1: unconnected-(D_RBOTTOM1-K-Pad1) -> ROW5
- D_RBOTTOM1 pad 2: unconnected-(D_RBOTTOM1-A-Pad2) -> Net-(D_RBOTTOM1-A)
- D_RCTRL1 pad 1: unconnected-(D_RCTRL1-K-Pad1) -> ROW5
- D_RCTRL1 pad 2: unconnected-(D_RCTRL1-A-Pad2) -> Net-(D_RCTRL1-A)
- D_RCURVE1 pad 1: Net-(D_EQ1-K) -> ROW2
- D_RCURVE1 pad 2: unconnected-(D_RCURVE1-A-Pad2) -> Net-(D_RCURVE1-A)
- D_REPEAT1 pad 1: ROW9 -> ROW7
- D_REPEAT1 pad 2: unconnected-(D_REPEAT1-A-Pad2) -> Net-(D_REPEAT1-A)
- D_RESUME1 pad 1: unconnected-(D_RESUME1-K-Pad1) -> ROW1
- D_RESUME1 pad 2: unconnected-(D_RESUME1-A-Pad2) -> Net-(D_RESUME1-A)
- D_RFN1 pad 1: ROW11 -> ROW6
- D_RFN1 pad 2: unconnected-(D_RFN1-A-Pad2) -> Net-(D_RFN1-A)
- D_RGREEK1 pad 1: ROW9 -> ROW4
- D_RGREEK1 pad 2: unconnected-(D_RGREEK1-A-Pad2) -> Net-(D_RGREEK1-A)
- D_RHYPER1 pad 1: unconnected-(D_RHYPER1-K-Pad1) -> ROW5
- D_RHYPER1 pad 2: unconnected-(D_RHYPER1-A-Pad2) -> Net-(D_RHYPER1-A)
- D_RMETA1 pad 1: unconnected-(D_RMETA1-K-Pad1) -> ROW5
- D_RMETA1 pad 2: unconnected-(D_RMETA1-A-Pad2) -> Net-(D_RMETA1-A)
- D_ROM_FOUR1 pad 1: ROW5 -> ROW8
- D_ROM_FOUR1 pad 2: unconnected-(D_ROM_FOUR1-A-Pad2) -> Net-(D_ROM_FOUR1-A)
- D_ROM_ONE1 pad 1: ROW1 -> ROW10
- D_ROM_THREE1 pad 1: ROW4 -> ROW2
- D_ROM_THREE1 pad 2: unconnected-(D_ROM_THREE1-A-Pad2) -> Net-(D_ROM_THREE1-A)
- D_ROM_TWO1 pad 1: ROW1 -> ROW2
- D_RPAREN1 pad 1: ROW5 -> ROW8
- D_RPAREN1 pad 2: unconnected-(D_RPAREN1-A-Pad2) -> Net-(D_RPAREN1-A)
- D_RSHIFT1 pad 1: ROW8 -> ROW4
- D_RSHIFT1 pad 2: unconnected-(D_RSHIFT1-A-Pad2) -> Net-(D_RSHIFT1-A)
- D_RSPACE1 pad 1: unconnected-(D_RSPACE1-K-Pad1) -> ROW5
- D_RSPACE1 pad 2: unconnected-(D_RSPACE1-A-Pad2) -> Net-(D_RSPACE1-A)
- D_RSUPER1 pad 1: unconnected-(D_RSUPER1-K-Pad1) -> ROW6
- D_RSUPER1 pad 2: unconnected-(D_RSUPER1-A-Pad2) -> Net-(D_RSUPER1-A)
- D_RTOP1 pad 1: ROW8 -> ROW4
- D_RTOP1 pad 2: unconnected-(D_RTOP1-A-Pad2) -> Net-(D_RTOP1-A)
- D_RUBOUT1 pad 1: ROW6 -> ROW7
- D_S1 pad 1: ROW6 -> ROW7
- D_S1 pad 2: unconnected-(D_S1-A-Pad2) -> Net-(D_S1-A)
- D_SEMICOLON1 pad 2: unconnected-(D_SEMICOLON1-A-Pad2) -> Net-(D_SEMICOLON1-A)
- D_SEVEN1 pad 1: ROW1 -> ROW10
- D_SIX1 pad 1: ROW1 -> ROW2
- D_SLASH1 pad 1: ROW9 -> ROW6
- D_SLASH1 pad 2: unconnected-(D_SLASH1-A-Pad2) -> Net-(D_SLASH1-A)
- D_STATUS1 pad 1: Net-(D_LCURVE1-K) -> ROW10
- D_STATUS1 pad 2: unconnected-(D_STATUS1-A-Pad2) -> Net-(D_STATUS1-A)
- D_STOP_OUTPUT1 pad 1: unconnected-(D_STOP_OUTPUT1-K-Pad1) -> ROW1
- D_STOP_OUTPUT1 pad 2: unconnected-(D_STOP_OUTPUT1-A-Pad2) -> Net-(D_STOP_OUTPUT1-A)
- D_SYSTEM1 pad 1: ROW1 -> ROW10
- D_T1 pad 1: ROW4 -> ROW2
- D_T1 pad 2: unconnected-(D_T1-A-Pad2) -> Net-(D_T1-A)
- D_TAB1 pad 1: ROW5 -> ROW8
- D_THREE1 pad 1: ROW1 -> ROW10
- D_THUMB_DOWN1 pad 1: Net-(D_LCURVE1-K) -> ROW10
- D_THUMB_DOWN1 pad 2: unconnected-(D_THUMB_DOWN1-A-Pad2) -> Net-(D_THUMB_DOWN1-A)
- D_THUMB_LEFT1 pad 1: ROW5 -> ROW3
- D_THUMB_LEFT1 pad 2: unconnected-(D_THUMB_LEFT1-A-Pad2) -> Net-(D_THUMB_LEFT1-A)
- D_THUMB_RIGHT1 pad 1: ROW4 -> ROW2
- D_THUMB_RIGHT1 pad 2: unconnected-(D_THUMB_RIGHT1-A-Pad2) -> Net-(D_THUMB_RIGHT1-A)
- D_THUMB_UP1 pad 1: Net-(D_EQ1-K) -> ROW2
- D_THUMB_UP1 pad 2: unconnected-(D_THUMB_UP1-A-Pad2) -> Net-(D_THUMB_UP1-A)
- D_TWO1 pad 1: ROW1 -> ROW2
- D_U1 pad 1: ROW4 -> ROW2
- D_U1 pad 2: unconnected-(D_U1-A-Pad2) -> Net-(D_U1-A)
- D_V1 pad 1: ROW9 -> ROW6
- D_W1 pad 1: ROW5 -> ROW8
- D_X1 pad 1: ROW9 -> ROW6
- D_X1 pad 2: unconnected-(D_X1-A-Pad2) -> Net-(D_X1-A)
- D_Y1 pad 1: ROW5 -> ROW8
- D_Y1 pad 2: unconnected-(D_Y1-A-Pad2) -> Net-(D_Y1-A)
- D_Z1 pad 1: ROW8 -> ROW4
- D_ZERO1 pad 1: Net-(D_EQ1-K) -> ROW2
- D_ZERO1 pad 2: unconnected-(D_ZERO1-A-Pad2) -> Net-(D_ZERO1-A)
- S_ABORT18 pad 1: COL8 -> COL9
- S_BACKSLASH1 pad 1: COL10 -> COL9
- S_BREAK1 pad 1: COL9 -> COL10
- S_COMMA1 pad 1: COL7 -> COL6
- S_DOT1 pad 1: COL8 -> COL7
- S_EQ1 pad 1: COL9 -> COL8
- S_K1 pad 1: COL7 -> COL6
- S_L1 pad 1: COL8 -> unconnected-(S_L1-in-Pad1)
- S_LINE1 pad 1: COL10 -> COL9
- S_P1 pad 1: COL8 -> COL7
- S_QUOTE1 pad 1: COL9 -> COL8
- S_RBOTTOM1 pad 1: COL7 -> COL8
- S_RCURVE1 pad 1: COL10 -> COL9
- S_REPEAT1 pad 1: COL11 -> COL10
- S_RESUME1 pad 1: COL10 -> COL11
- S_RETURN1 pad 1: COL9 -> COL8
- S_RETURN1 pad 2: Net-(D_RETURN1-A) -> unconnected-(S_RETURN1-out-Pad2)
- S_RGREEK1 pad 1: COL10 -> COL9
- S_RPAREN1 pad 1: COL9 -> COL8
- S_RSHIFT1 pad 1: COL9 -> COL8
- S_RSUPER1 pad 1: COL11 -> COL10
- S_SEMICOLON1 pad 1: COL8 -> COL7
- S_SLASH1 pad 1: COL8 -> COL7
- S_STOP_OUTPUT1 pad 1: COL7 -> COL8
- S_THUMB_LEFT1 pad 1: COL11 -> COL10
- S_THUMB_UP1 pad 1: COL11 -> COL10
- S_ZERO1 pad 1: COL8 -> COL7
Routing:
- net ROW11: track 796.1 -> 0.00 mm
- net ROW2: track 0.00 -> 782.3 mm
- net ROW5: track 548.4 -> 1229.6 mm
- net ROW9: track 596.5 -> 0.00 mm
- net (no net): track 0.10 -> 486.9 mm
- net ROW6: track 470.5 -> 71.3 mm
- net ROW7: track 523.4 -> 910.8 mm
- net ROW10: track 815.7 -> 458.6 mm, vias 2 -> 0
- net Net-(D_EQ1-K): track 261.0 -> 0.00 mm
- net COL6: track 365.0 -> 167.8 mm
- net ROW1: track 477.4 -> 381.0 mm
- net ROW8: track 500.9 -> 554.5 mm
- net ROW4: track 481.3 -> 433.9 mm
- net ROW3: track 0.00 -> 46.0 mm
- net COL7: track 392.7 -> 354.8 mm
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
Commit message: wip: handwiring
Parts:
- S_BACKSLASH1, S_EQ1, S_MINUS1, S_REPEAT1, S_RFN1: footprint Button_Switch_Keyboard:SWMXK_1.00u -> Button_Switch_Keyboard:SWMXK_1.50u
- S_LINE1, S_RBACK1, S_RBOTTOM1: footprint Button_Switch_Keyboard:SWMXK_1.00u -> Button_Switch_Keyboard:SWMXK_1.25u
- S_LSPACE1: footprint Button_Switch_Keyboard:SWMXK_1.00u -> Button_Switch_Keyboard:SWMXK_2.75u
- S_QUOTE1: footprint Button_Switch_Keyboard:SWMXK_2.00u -> Button_Switch_Keyboard:SWMXK_1.00u
- S_RCTRL1: footprint Button_Switch_Keyboard:SWMXK_1.00u -> Button_Switch_Keyboard:SWMXK_1.75u
- S_RSHIFT1: footprint Button_Switch_Keyboard:SWMXK_1.50u -> Button_Switch_Keyboard:SWMXK_2.25u
- S_RSPACE1: footprint Button_Switch_Keyboard:SWMXK_1.00u -> Button_Switch_Keyboard:SWMXK_2.25u
- S_TAB1: footprint Button_Switch_Keyboard:SWMXK_1.75u -> Button_Switch_Keyboard:SWMXK_1.50u
- moved D_CALL1 16.2 mm to (449.4, 35.6), turned to 90 degrees
- moved D_LHYPER1 15.2 mm to (25.6, 129.8), turned to 90 degrees
- moved D_LMETA1 15.2 mm to (82.7, 129.8), turned to 90 degrees
- moved D_ROM_FOUR1 15.2 mm to (39.9, 72.7), turned to 90 degrees
- moved D_TAB1 15.2 mm to (101.8, 72.7), turned to 90 degrees
- moved D_COLON1 15.2 mm to (97.0, 53.6), turned to 90 degrees
- moved D_ROM_TWO1 15.2 mm to (40.0, 53.6), turned to 90 degrees
- moved D_CAPS_LOCK1 15.2 mm to (20.8, 110.8), turned to 90 degrees
- moved D_LGREEK1 15.2 mm to (73.2, 110.8), turned to 90 degrees
- moved D_RUBOUT1 15.2 mm to (104.2, 91.7), turned to 90 degrees
- moved D_LSPACE1 13.5 mm to (213.2, 129.8), turned to 90 degrees
- moved D_RSPACE1 13.5 mm to (261.0, 129.8), turned to 90 degrees
- moved D_RSHIFT1 13.3 mm to (351.1, 110.8), turned to 90 degrees
- moved D_THUMB_LEFT1 13.3 mm to (439.7, 72.7), turned to 90 degrees
- moved D_RBOTTOM1 13.3 mm to (285.0, 129.8), turned to 90 degrees
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Connections:
- D_CALL1 pad 1: ROW2 -> ROW9
- D_COLON1 pad 1: ROW2 -> ROW9
- D_EIGHT1 pad 1: ROW2 -> ROW9
- D_EQ1 pad 1: ROW2 -> ROW9
- D_FOUR1 pad 1: ROW2 -> ROW9
- D_RCURVE1 pad 1: ROW2 -> ROW9
- D_RETURN1 pad 2: unconnected-(D_RETURN1-A-Pad2) -> Net-(D_RETURN1-A)
- D_ROM_TWO1 pad 1: ROW2 -> ROW9
- D_SIX1 pad 1: ROW2 -> ROW9
- D_THUMB_UP1 pad 1: ROW2 -> ROW9
- D_TWO1 pad 1: ROW2 -> ROW9
- D_ZERO1 pad 1: ROW2 -> ROW9
- S_L1 pad 1: unconnected-(S_L1-in-Pad1) -> COL7
- S_RETURN1 pad 2: unconnected-(S_RETURN1-out-Pad2) -> Net-(D_RETURN1-A)
Routing:
- net ROW5: track 1229.6 -> 429.8 mm
- net ROW7: track 910.8 -> 398.1 mm
- net (no net): track 486.9 -> 0.26 mm
- net ROW9: track 0.00 -> 453.6 mm
- net ROW3: track 46.0 -> 423.1 mm
- net ROW2: track 782.3 -> 438.2 mm
- net ROW6: track 71.3 -> 414.0 mm, vias 0 -> 2
- net ROW8: track 554.5 -> 338.1 mm
- net COL7: track 354.8 -> 240.3 mm
- net COL6: track 167.8 -> 251.3 mm
- net COL11: track 263.2 -> 210.5 mm
- net COL10: track 220.8 -> 266.1 mm, vias 6 -> 0
- net COL8: track 231.1 -> 260.8 mm
- net COL2: track 234.2 -> 259.6 mm, vias 10 -> 0
- net ROW10: track 458.6 -> 438.2 mm
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
Commit message: upd: diode footprint
Parts:
- D_A1, D_ABORT1, D_ALTLOCK1, D_ALTMODE1, D_B1, D_BACK1, D_BACKSLASH1, D_BACKTICK1, D_BREAK1, D_C1, D_CALL1, D_CAPS_LOCK1, D_CLEAR_INPUT1, D_CLEAR_SCREEN1, D_COLON1, D_COMMA1, D_D1, D_DELETE1, D_DOT1, D_E1, D_EIGHT1, D_END1, D_EQ1, D_F1, D_FIVE1, D_FOUR1, D_G1, D_H1, D_HELP1, D_HOLD_OUTPUT1, D_I_1, D_J1, D_K1, D_L1, D_LBACK1, D_LBOTTOM1, D_LCTRL1, D_LCURVE1, D_LGREEK1, D_LHYPER1, D_LINE1, D_LMETA1, D_LPAREN1, D_LSHIFT1, D_LSPACE1, D_LSUPER1, D_LTOP1, D_M1, D_MACRO1, D_MINUS1, D_MODE_LOCK1, D_N1, D_NETWORK1, D_NINE1, D_O1, D_ONE1, D_OVER_STRIKE1, D_P1, D_Q1, D_QUOTE1, D_QUOTE_MOD1, D_R1, D_RBOTTOM1, D_RCTRL1, D_RCURVE1, D_REPEAT1, D_RESUME1, D_RETURN1, D_RFN1, D_RGREEK1, D_RHYPER1, D_RMETA1, D_ROM_FOUR1, D_ROM_ONE1, D_ROM_THREE1, D_ROM_TWO1, D_RPAREN1, D_RSHIFT1, D_RSPACE1, D_RSUPER1, D_RTOP1, D_RUBOUT1, D_S1, D_SEMICOLON1, D_SEVEN1, D_SIX1, D_SLASH1, D_STATUS1, D_STOP_OUTPUT1, D_SYSTEM1, D_T1, D_TAB1, D_TERMINAL1, D_THREE1, D_THUMB_DOWN1, D_THUMB_LEFT1, D_THUMB_RIGHT1, D_THUMB_UP1, D_TWO1, D_U1, D_V1, D_W1, D_X1, D_Y1, D_Z1, D_ZERO1: footprint Diode_THT:D_DO-41_SOD81_P7.62mm_Horizontal -> Button_Switch_Keyboard:D_P7.62mm

Commit message: upd: RPI footprint
Parts:
- U101: footprint RPI:RPi_Pico_SMD_TH -> Button_Switch_Keyboard:RPi_Pico_SMD_TH

Commit message: wip: renew
Parts:
- moved U101 43.2 mm to (419.7, 171.5), turned to -90 degrees
- moved D_RSPACE1 26.1 mm to (235.3, 134.4)
- moved D_LSPACE1 24.5 mm to (189.1, 134.3)
- moved D_RESUME1 18.9 mm to (405.0, 37.1), turned to 90 degrees
- moved D_TERMINAL1 18.3 mm to (64.0, 37.1), turned to 90 degrees
- moved D_CLEAR_INPUT1 17.8 mm to (182.8, 37.1), turned to 90 degrees
- moved D_ABORT1 17.8 mm to (335.1, 37.1), turned to 90 degrees
- moved D_BREAK1 17.8 mm to (373.2, 37.1), turned to 90 degrees
- moved D_CLEAR_SCREEN1 17.8 mm to (220.9, 37.1), turned to 90 degrees
- moved D_HOLD_OUTPUT1 17.8 mm to (259.0, 37.1), turned to 90 degrees
- moved D_MACRO1 17.8 mm to (30.4, 37.1), turned to 90 degrees
- moved D_OVER_STRIKE1 17.8 mm to (144.7, 37.1), turned to 90 degrees
- moved D_QUOTE_MOD1 17.8 mm to (106.6, 37.1), turned to 90 degrees
- moved D_STOP_OUTPUT1 17.8 mm to (297.0, 37.1), turned to 90 degrees
- moved D_LBACK1 4.46 mm to (142.1, 134.3)
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Connections:
- D_A1 pad 1: ROW3 -> ROW4
- D_ALTLOCK1 pad 1: ROW4 -> ROW5
- D_ALTMODE1 pad 1: ROW3 -> ROW4
- D_B1 pad 1: ROW4 -> ROW5
- D_BACK1 pad 1: ROW6 -> ROW7
- D_BACKSLASH1 pad 1: ROW8 -> ROW9
- D_BACKTICK1 pad 1: ROW2 -> ROW3
- D_C1 pad 1: ROW4 -> ROW5
- D_CALL1 pad 1: ROW9 -> ROW10
- D_CAPS_LOCK1 pad 1: ROW4 -> ROW5
- D_COLON1 pad 1: ROW9 -> ROW10
- D_COMMA1 pad 1: ROW6 -> ROW7
- D_D1 pad 1: ROW3 -> ROW4
- D_DELETE1 pad 1: ROW2 -> ROW3
- D_DOT1 pad 1: ROW4 -> ROW5
- D_E1 pad 1: ROW2 -> ROW3
- D_EIGHT1 pad 1: ROW9 -> ROW10
- D_END1 pad 1: ROW3 -> ROW4
- D_EQ1 pad 1: ROW9 -> ROW10
- D_F1 pad 1: ROW7 -> ROW8
- D_FIVE1 pad 1: ROW10 -> ROW2
- D_FOUR1 pad 1: ROW9 -> ROW10
- D_G1 pad 1: ROW3 -> ROW4
- D_H1 pad 1: ROW7 -> ROW8
- D_HELP1 pad 1: ROW3 -> ROW4
- D_I_1 pad 1: ROW8 -> ROW9
- D_J1 pad 1: ROW3 -> ROW4
- D_K1 pad 1: ROW7 -> ROW8
- D_L1 pad 1: ROW3 -> ROW4
- D_LBACK1 pad 1: ROW5 -> ROW6
- D_LBOTTOM1 pad 1: ROW5 -> ROW6
- D_LCTRL1 pad 1: ROW5 -> ROW6
- D_LCURVE1 pad 1: ROW10 -> ROW2
- D_LGREEK1 pad 1: ROW4 -> ROW5
- D_LHYPER1 pad 1: ROW5 -> ROW6
- D_LINE1 pad 1: ROW3 -> ROW4
- D_LMETA1 pad 1: ROW5 -> ROW6
- D_LPAREN1 pad 1: ROW2 -> ROW3
- D_LSHIFT1 pad 1: ROW6 -> ROW7
- D_LSPACE1 pad 1: ROW5 -> ROW6
- D_LSUPER1 pad 1: ROW6 -> ROW7
- D_LTOP1 pad 1: ROW7 -> ROW8
- D_M1 pad 1: ROW4 -> ROW5
- D_MINUS1 pad 1: ROW10 -> ROW2
- D_MODE_LOCK1 pad 1: ROW3 -> ROW4
- D_N1 pad 1: ROW6 -> ROW7
- D_NETWORK1 pad 1: ROW2 -> ROW3
- D_NINE1 pad 1: ROW10 -> ROW2
- D_O1 pad 1: ROW2 -> ROW3
- D_ONE1 pad 1: ROW10 -> ROW2
- D_P1 pad 1: ROW8 -> ROW9
- D_Q1 pad 1: ROW2 -> ROW3
- D_QUOTE1 pad 1: ROW3 -> ROW4
- D_R1 pad 1: ROW8 -> ROW9
- D_RBOTTOM1 pad 1: ROW5 -> ROW6
- D_RCTRL1 pad 1: ROW5 -> ROW6
- D_RCURVE1 pad 1: ROW9 -> ROW10
- D_REPEAT1 pad 1: ROW7 -> ROW8
- D_RETURN1 pad 1: ROW7 -> ROW8
- D_RFN1 pad 1: ROW6 -> ROW7
- D_RGREEK1 pad 1: ROW4 -> ROW5
- D_RHYPER1 pad 1: ROW5 -> ROW6
- D_RMETA1 pad 1: ROW5 -> ROW6
- D_ROM_FOUR1 pad 1: ROW8 -> ROW9
- D_ROM_ONE1 pad 1: ROW10 -> ROW2
- D_ROM_THREE1 pad 1: ROW2 -> ROW3
- D_ROM_TWO1 pad 1: ROW9 -> ROW10
- D_RPAREN1 pad 1: ROW8 -> ROW9
- D_RSHIFT1 pad 1: ROW4 -> ROW5
- D_RSPACE1 pad 1: ROW5 -> ROW6
- D_RSUPER1 pad 1: ROW6 -> ROW7
- D_RTOP1 pad 1: ROW4 -> ROW5
- D_RUBOUT1 pad 1: ROW7 -> ROW8
- D_S1 pad 1: ROW7 -> ROW8
- D_SEMICOLON1 pad 1: ROW7 -> ROW8
- D_SEVEN1 pad 1: ROW10 -> ROW2
- D_SIX1 pad 1: ROW9 -> ROW10
- D_SLASH1 pad 1: ROW6 -> ROW7
- D_STATUS1 pad 1: ROW10 -> ROW2
- D_SYSTEM1 pad 1: ROW10 -> ROW2
- D_T1 pad 1: ROW2 -> ROW3
- D_TAB1 pad 1: ROW8 -> ROW9
- D_THREE1 pad 1: ROW10 -> ROW2
- D_THUMB_DOWN1 pad 1: ROW10 -> ROW2
- D_THUMB_LEFT1 pad 1: ROW3 -> ROW9
- D_THUMB_RIGHT1 pad 1: ROW2 -> ROW3
- D_THUMB_UP1 pad 1: ROW9 -> ROW10
- D_TWO1 pad 1: ROW9 -> ROW10
- D_U1 pad 1: ROW2 -> ROW3
- D_V1 pad 1: ROW6 -> ROW7
- D_W1 pad 1: ROW8 -> ROW9
- D_X1 pad 1: ROW6 -> ROW7
- D_Y1 pad 1: ROW8 -> ROW9
- D_Z1 pad 1: ROW4 -> ROW5
- D_ZERO1 pad 1: ROW9 -> ROW10
Routing:
- net COL1: track 299.9 -> 430.1 mm
- net COL10: track 266.1 -> 381.6 mm
- net COL6: track 251.3 -> 342.5 mm
- net COL7: track 240.3 -> 326.3 mm
- net COL2: track 259.6 -> 340.4 mm
- net COL4: track 222.6 -> 298.7 mm
- net COL3: track 215.0 -> 288.5 mm
- net COL8: track 260.8 -> 334.3 mm
- net COL5: track 239.0 -> 310.0 mm
- net COL9: track 232.5 -> 296.2 mm
- net ROW8: track 338.1 -> 394.6 mm
- net ROW9: track 453.6 -> 399.8 mm
- net Net-(D_RSPACE1-A): track 23.8 -> 65.9 mm
- net Net-(D_LSPACE1-A): track 23.9 -> 62.9 mm
- net Net-(D_RSHIFT1-A): track 23.8 -> 53.4 mm
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Other:
- board size 473.2 x 186 mm -> 473.2 x 194.3 mm

Commit message: imp: vcc & gnd added
Connections:
- U101 pad 13: unconnected-(U101-GND-Pad13) -> GND
- U101 pad 18: unconnected-(U101-GND-Pad18) -> GND
- U101 pad 23: unconnected-(U101-GND-Pad23) -> GND
- U101 pad 28: unconnected-(U101-GND-Pad28) -> GND
- U101 pad 3: unconnected-(U101-GND-Pad3) -> GND
- U101 pad 38: unconnected-(U101-GND-Pad38) -> GND
- U101 pad 39: unconnected-(U101-VSYS-Pad39) -> VCC
- U101 pad 40: unconnected-(U101-VBUS-Pad40) -> VCC
