File: SpaceCadet.kicad_pcb (KiCad board)
At the start: 2 copper layers, 473.2 x 194.3 mm, 214 parts, among them U101 Pico

Commit message: wip: rpi pico on pcb
Parts:
- moved U101 360.8 mm to (58.9, 163.2), turned to 180 degrees
- moved D_RSPACE1 11.6 mm to (246.9, 133.9)
- moved D_BACKTICK1 10.2 mm to (364.4, 57.5)
- moved D_DOT1 10.2 mm to (302.4, 112.8)
- moved D_HELP1 10.2 mm to (459.8, 76.6)
- moved D_O1 10.2 mm to (288.2, 57.5)
- moved D_QUOTE1 10.2 mm to (331.1, 76.6)
- moved D_RHYPER1 10.2 mm to (464.4, 133.8)
- moved D_THUMB_UP1 10.2 mm to (449.9, 55.7)
- moved D_ZERO1 10.2 mm to (297.7, 55.7)
- moved S_ABORT18 10.2 mm to (356.6, 23.9)
- moved S_ALTLOCK1 10.2 mm to (480.4, 100.1)
- moved S_BACKSLASH1 10.2 mm to (399.4, 62.0)
- moved S_BACKTICK1 10.2 mm to (375.6, 62.0)
- moved S_DOT1 10.2 mm to (313.7, 100.1)
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Connections:
- U101 pad 10: unconnected-(U101-GPIO7-Pad10) -> COL9
- U101 pad 11: unconnected-(U101-GPIO8-Pad11) -> COL8
- U101 pad 12: unconnected-(U101-GPIO9-Pad12) -> COL7
- U101 pad 13: GND -> unconnected-(U101-GND-Pad13)
- U101 pad 14: unconnected-(U101-GPIO10-Pad14) -> COL6
- U101 pad 15: unconnected-(U101-GPIO11-Pad15) -> COL5
- U101 pad 16: unconnected-(U101-GPIO12-Pad16) -> COL4
- U101 pad 17: unconnected-(U101-GPIO13-Pad17) -> COL3
- U101 pad 18: GND -> unconnected-(U101-GND-Pad18)
- U101 pad 19: unconnected-(U101-GPIO14-Pad19) -> COL2
- U101 pad 20: unconnected-(U101-GPIO15-Pad20) -> COL1
- U101 pad 21: unconnected-(U101-GPIO16-Pad21) -> ROW6
- U101 pad 22: unconnected-(U101-GPIO17-Pad22) -> ROW7
- U101 pad 23: GND -> unconnected-(U101-GND-Pad23)
- U101 pad 24: unconnected-(U101-GPIO18-Pad24) -> ROW5
- U101 pad 25: unconnected-(U101-GPIO19-Pad25) -> ROW8
- U101 pad 26: unconnected-(U101-GPIO20-Pad26) -> ROW4
- U101 pad 27: unconnected-(U101-GPIO21-Pad27) -> ROW9
- U101 pad 28: GND -> unconnected-(U101-GND-Pad28)
- U101 pad 29: unconnected-(U101-GPIO22-Pad29) -> ROW3
- U101 pad 3: GND -> unconnected-(U101-GND-Pad3)
- U101 pad 31: unconnected-(U101-GPIO26_ADC0-Pad31) -> ROW10
- U101 pad 32: unconnected-(U101-GPIO27_ADC1-Pad32) -> ROW2
- U101 pad 34: unconnected-(U101-GPIO28_ADC2-Pad34) -> ROW1
- U101 pad 38: GND -> unconnected-(U101-GND-Pad38)
- U101 pad 7: unconnected-(U101-GPIO5-Pad7) -> COL11
- U101 pad 9: unconnected-(U101-GPIO6-Pad9) -> COL10
Routing:
- net COL11: track 221.7 -> 682.3 mm
- net COL10: track 381.6 -> 783.6 mm, vias 0 -> 1
- net COL9: track 296.2 -> 680.3 mm, vias 0 -> 1
- net COL8: track 334.3 -> 655.6 mm, vias 0 -> 1
- net COL7: track 326.3 -> 598.8 mm, vias 0 -> 1
- net COL6: track 342.5 -> 560.0 mm, vias 0 -> 1
- net ROW1: track 374.6 -> 570.2 mm
- net ROW2: track 438.2 -> 612.4 mm
- net COL5: track 310.0 -> 479.4 mm, vias 0 -> 1
- net ROW10: track 432.7 -> 601.5 mm
- net ROW3: track 438.3 -> 577.7 mm
- net COL4: track 298.7 -> 437.6 mm, vias 0 -> 1
- net ROW9: track 399.8 -> 530.7 mm
- net ROW4: track 419.3 -> 531.8 mm
- net ROW8: track 394.6 -> 497.2 mm
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Other:
- board size 473.2 x 194.3 mm -> 489.8 x 194.3 mm

Commit message: wip: pri fully connected with test points
Parts:
- added TP101: TestPoint, TestPoint:TestPoint_THTPad_2.0x2.0mm_Drill1.0mm, F.Cu at (37.3, 189.8)
- added TP102: TestPoint, TestPoint:TestPoint_THTPad_2.0x2.0mm_Drill1.0mm, F.Cu at (32.4, 194.8)
- added TP103: TestPoint, TestPoint:TestPoint_THTPad_2.0x2.0mm_Drill1.0mm, F.Cu at (105.1, 194.8)
- added TP104: TestPoint, TestPoint:TestPoint_THTPad_2.0x2.0mm_Drill1.0mm, F.Cu at (115.7, 192.3)
- added TP105: TestPoint, TestPoint:TestPoint_THTPad_2.0x2.0mm_Drill1.0mm, F.Cu at (105.1, 187.2)
- added TP106: TestPoint, TestPoint:TestPoint_THTPad_2.0x2.0mm_Drill1.0mm, F.Cu at (115.7, 184.6)
- added TP107: TestPoint, TestPoint:TestPoint_THTPad_2.0x2.0mm_Drill1.0mm, F.Cu at (105.1, 182.1)
- added TP108: TestPoint, TestPoint:TestPoint_THTPad_2.0x2.0mm_Drill1.0mm, F.Cu at (16.9, 187.2)
- added TP109: TestPoint, TestPoint:TestPoint_THTPad_2.0x2.0mm_Drill1.0mm, F.Cu at (24.2, 184.6)
- added TP110: TestPoint, TestPoint:TestPoint_THTPad_2.0x2.0mm_Drill1.0mm, F.Cu at (16.9, 182.1)
- added TP111: TestPoint, TestPoint:TestPoint_THTPad_2.0x2.0mm_Drill1.0mm, F.Cu at (24.6, 169.4)
- added TP112: TestPoint, TestPoint:TestPoint_THTPad_2.0x2.0mm_Drill1.0mm, F.Cu at (61.5, 141.0)
- added TP113: TestPoint, TestPoint:TestPoint_THTPad_2.0x2.0mm_Drill1.0mm, F.Cu at (58.9, 136.4)
- added TP114: TestPoint, TestPoint:TestPoint_THTPad_2.0x2.0mm_Drill1.0mm, F.Cu at (56.4, 141.0)
- added TP201: TestPoint, TestPoint:TestPoint_THTPad_2.0x2.0mm_Drill1.0mm, F.Cu at (40.6, 179.6)
- added TP202: TestPoint, TestPoint:TestPoint_THTPad_2.0x2.0mm_Drill1.0mm, F.Cu at (35.8, 174.6)
- added TP203: TestPoint, TestPoint:TestPoint_THTPad_2.0x2.0mm_Drill1.0mm, F.Cu at (40.6, 172.1)
- added TP204: TestPoint, TestPoint:TestPoint_THTPad_2.0x2.0mm_Drill1.0mm, F.Cu at (35.8, 166.9)
- added TP205: TestPoint, TestPoint:TestPoint_THTPad_2.0x2.0mm_Drill1.0mm, F.Cu at (40.6, 161.9)
- added TP206: TestPoint, TestPoint:TestPoint_THTPad_2.0x2.0mm_Drill1.0mm, F.Cu at (35.8, 159.3)
- added TP207: TestPoint, TestPoint:TestPoint_THTPad_2.0x2.0mm_Drill1.0mm, F.Cu at (40.6, 156.7)
- added TP208: TestPoint, TestPoint:TestPoint_THTPad_2.0x2.0mm_Drill1.0mm, F.Cu at (35.8, 154.2)
- added TP209: TestPoint, TestPoint:TestPoint_THTPad_2.0x2.0mm_Drill1.0mm, F.Cu at (40.6, 149.1)
- added TP210: TestPoint, TestPoint:TestPoint_THTPad_2.0x2.0mm_Drill1.0mm, F.Cu at (35.8, 146.5)
- added TP211: TestPoint, TestPoint:TestPoint_THTPad_2.0x2.0mm_Drill1.0mm, F.Cu at (83.3, 179.5)
- added TP212: TestPoint, TestPoint:TestPoint_THTPad_2.0x2.0mm_Drill1.0mm, F.Cu at (93.9, 174.5)
- added TP213: TestPoint, TestPoint:TestPoint_THTPad_2.0x2.0mm_Drill1.0mm, F.Cu at (83.3, 171.9)
- added TP214: TestPoint, TestPoint:TestPoint_THTPad_2.0x2.0mm_Drill1.0mm, F.Cu at (93.9, 169.4)
- added TP215: TestPoint, TestPoint:TestPoint_THTPad_2.0x2.0mm_Drill1.0mm, F.Cu at (83.3, 166.8)
- added TP216: TestPoint, TestPoint:TestPoint_THTPad_2.0x2.0mm_Drill1.0mm, F.Cu at (93.9, 161.8)
- added TP217: TestPoint, TestPoint:TestPoint_THTPad_2.0x2.0mm_Drill1.0mm, F.Cu at (83.3, 159.2)
- added TP218: TestPoint, TestPoint:TestPoint_THTPad_2.0x2.0mm_Drill1.0mm, F.Cu at (93.9, 156.6)
- added TP219: TestPoint, TestPoint:TestPoint_THTPad_2.0x2.0mm_Drill1.0mm, F.Cu at (83.3, 154.2)
- added TP220: TestPoint, TestPoint:TestPoint_THTPad_2.0x2.0mm_Drill1.0mm, F.Cu at (93.9, 149.1)
- added TP221: TestPoint, TestPoint:TestPoint_THTPad_2.0x2.0mm_Drill1.0mm, F.Cu at (83.3, 146.6)
- moved U101 7.49 mm to (58.9, 170.7)
Connections:
- net VCC renamed VSS
- U101 pad 1: unconnected-(U101-GPIO0-Pad1) -> Net-(U101-GPIO0)
- U101 pad 13: unconnected-(U101-GND-Pad13) -> GND
- U101 pad 18: unconnected-(U101-GND-Pad18) -> GND
- U101 pad 2: unconnected-(U101-GPIO1-Pad2) -> Net-(U101-GPIO1)
- U101 pad 23: unconnected-(U101-GND-Pad23) -> GND
- U101 pad 28: unconnected-(U101-GND-Pad28) -> GND
- U101 pad 3: unconnected-(U101-GND-Pad3) -> GND
- U101 pad 30: unconnected-(U101-RUN-Pad30) -> Net-(U101-RUN)
- U101 pad 33: unconnected-(U101-AGND-Pad33) -> GND
- U101 pad 35: unconnected-(U101-ADC_VREF-Pad35) -> Net-(U101-ADC_VREF)
- U101 pad 36: unconnected-(U101-3V3-Pad36) -> Net-(U101-3V3)
- U101 pad 37: unconnected-(U101-3V3_EN-Pad37) -> Net-(U101-3V3_EN)
- U101 pad 38: unconnected-(U101-GND-Pad38) -> GND
- U101 pad 4: unconnected-(U101-GPIO2-Pad4) -> Net-(U101-GPIO2)
- U101 pad 41: unconnected-(U101-SWCLK-Pad41) -> Net-(U101-SWCLK)
- U101 pad 42: unconnected-(U101-GND-Pad42) -> Net-(TP113-Pad1)
- U101 pad 43: unconnected-(U101-SWDIO-Pad43) -> Net-(U101-SWDIO)
- U101 pad 5: unconnected-(U101-GPIO3-Pad5) -> Net-(U101-GPIO3)
- U101 pad 6: unconnected-(U101-GPIO4-Pad6) -> Net-(U101-GPIO4)
- U101 pad 8: unconnected-(U101-GND-Pad8) -> GND
Routing:
- net COL5: track 479.4 -> 352.1 mm
- net GND: track 0.00 -> 122.0 mm
- net Net-(U101-GPIO1): track 0.00 -> 47.9 mm
- net Net-(U101-GPIO3): track 0.00 -> 47.9 mm
- net Net-(U101-GPIO4): track 0.00 -> 37.3 mm
- net Net-(U101-GPIO0): track 0.00 -> 37.3 mm
- net Net-(U101-GPIO2): track 0.00 -> 37.3 mm
- net Net-(U101-3V3_EN): track 0.00 -> 33.1 mm
- net Net-(U101-ADC_VREF): track 0.00 -> 33.1 mm
- net VSS: track 0.00 -> 28.8 mm
- net Net-(U101-3V3): track 0.00 -> 25.9 mm
- net Net-(U101-RUN): track 0.00 -> 25.5 mm
- net ROW6: track 440.4 -> 455.8 mm
- net Net-(TP113-Pad1): track 0.00 -> 10.4 mm
- net ROW10: track 601.5 -> 609.2 mm
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
Commit message: fix: unconnected
Routing:
- net COL5: track 352.1 -> 486.9 mm
- net COL10: track 791.1 -> 796.8 mm
Changed lines of the file:
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@@
+	)
+	(segment
+		(start 83.277587 159.208671)
+		(end 196.088 159.208671)
+		(width 0.75)
+		(layer "B.Cu")
+		(net 91)
 	)
 	(segment
@@
 		(start 232.76101 42.959997)
 		(end 236.34701 42.959997)
+		(width 0.75)
+		(layer "B.Cu")
+		(net 91)
+	)
+	(segment
+		(start 196.088 159.208671)
+		(end 196.088 137.16)
 		(width 0.75)
 		(layer "B.Cu")
@@
 		(end 487.172 81.034994)
 		(width 0.75)
-		(layer "B.Cu")
-		(net 99)
-	)
-	(segment
-		(start 489.206058 24.06)
-		(end 489.166058 24.02)
-		(width 0.5)
 		(layer "B.Cu")
 		(net 99)
@@
 	)
 	(segment
+		(start 418.49859 119.160004)
+		(end 422.08459 119.160004)
+		(width 0.75)
+		(layer "B.Cu")
+		(net 102)
+	)
+	(segment
 		(start 394.68599 23.91)
 		(end 398.27199 23.91)
@@
 	)
 	(segment
+		(start 424.206058 116.59)
+		(end 424.206058 119.135004)
+		(width 0.75)
+		(layer "B.Cu")
+		(net 102)
+	)
+	(segment
 		(start 432.205874 81.64)
 		(end 432.78588 81.059994)
@@
 	)
 	(segment
+		(start 422.08459 119.160004)
+		(end 422.08459 119.135004)
+		(width 0.75)
+		(layer "B.Cu")
+		(net 102)
+	)
+	(segment
 		(start 461.36092 42.959997)
 		(end 464.94692 42.959997)
@@
 	)
 	(segment
+		(start 424.206058 119.135004)
+		(end 422.08459 119.135004)
+		(width 0.75)
+		(layer "B.Cu")
+		(net 102)
+	)
+	(segment
 		(start 93.93699 174.498517)
 		(end 425.196 174.498517)
 		(width 0.75)
 		(layer "B.Cu")
-		(net 102)
-	)
-	(segment
-		(start 424.206058 116.59)
-		(end 424.206058 119.160004)
-		(width 0.75)
-		(layer "B.Cu")

Commit message: imp: via test points pcb
Parts:
- added REF**: TestPoint_THTPad_2.0x2.0mm_Drill1.0mm, TestPoint:TestPoint_THTPad_2.0x2.0mm_Drill1.0mm, F.Cu at (243.8, 137.2)
- added REF**: TestPoint_THTPad_2.0x2.0mm_Drill1.0mm, TestPoint:TestPoint_THTPad_2.0x2.0mm_Drill1.0mm, F.Cu at (142.2, 137.2)
- added REF**: TestPoint_THTPad_2.0x2.0mm_Drill1.0mm, TestPoint:TestPoint_THTPad_2.0x2.0mm_Drill1.0mm, F.Cu at (398.3, 137.2)
- added REF**: TestPoint_THTPad_2.0x2.0mm_Drill1.0mm, TestPoint:TestPoint_THTPad_2.0x2.0mm_Drill1.0mm, F.Cu at (292.6, 137.2)
- added REF**: TestPoint_THTPad_2.0x2.0mm_Drill1.0mm, TestPoint:TestPoint_THTPad_2.0x2.0mm_Drill1.0mm, F.Cu at (196.1, 137.2)
- added REF**: TestPoint_THTPad_2.0x2.0mm_Drill1.0mm, TestPoint:TestPoint_THTPad_2.0x2.0mm_Drill1.0mm, F.Cu at (111.8, 137.2)
- added REF**: TestPoint_THTPad_2.0x2.0mm_Drill1.0mm, TestPoint:TestPoint_THTPad_2.0x2.0mm_Drill1.0mm, F.Cu at (73.3, 114.6)
- added REF**: TestPoint_THTPad_2.0x2.0mm_Drill1.0mm, TestPoint:TestPoint_THTPad_2.0x2.0mm_Drill1.0mm, F.Cu at (170.2, 137.2)
- added REF**: TestPoint_THTPad_2.0x2.0mm_Drill1.0mm, TestPoint:TestPoint_THTPad_2.0x2.0mm_Drill1.0mm, F.Cu at (73.3, 95.7)
- added REF**: TestPoint_THTPad_2.0x2.0mm_Drill1.0mm, TestPoint:TestPoint_THTPad_2.0x2.0mm_Drill1.0mm, F.Cu at (338.3, 137.2)
- added REF**: TestPoint_THTPad_2.0x2.0mm_Drill1.0mm, TestPoint:TestPoint_THTPad_2.0x2.0mm_Drill1.0mm, F.Cu at (425.2, 137.2)
Routing:
- net ROW7: vias 2 -> 4
- net COL8: vias 1 -> 2
- net COL7: vias 1 -> 2
- net COL6: vias 1 -> 2
- net COL5: vias 1 -> 2
- net COL4: vias 1 -> 2
- net COL3: vias 1 -> 2
- net COL2: vias 1 -> 2
- net COL10: vias 1 -> 2

Commit message: test: for gbr
Parts:
- added REF**: DIP-8_W7.62mm_LongPads, Package_DIP:DIP-8_W7.62mm_LongPads, F.Cu at (445.5, 25.2)
Routing:
- net (no net): track 0.09 -> 75.5 mm
Other:
- board size 489.8 x 194.3 mm -> 487.2 x 189.4 mm

Commit message: fix: bigger borders
Parts:
- removed the REF** at (445.5, 25.2)
Routing:
- net (no net): track 75.5 -> 0.09 mm
Other:
- board size 487.2 x 189.4 mm -> 493.6 x 197 mm
